File: PCB.sch (EAGLE design)
At the start: 40 parts, among them IC1 STM32F407VGT6, IC2 LD1117S33CTR, IC3 LTC6811-1, IC6 LTC6811-1, IC7 LTC6811-1, Q1 IRLML5203, Q2 IRLML5203, U1 OKI-78SR-5_1.5-W36-C, U2 OKI-78SR-5_1.5-W36-C, U3 OKI-78SR-5_1.5-W36-C, U4 OKI-78SR-5_1.5-W36-C, X4 B4B-ZR, X5 B4B-ZR, X6 B4B-ZR

Commit message: update pcb
Parts:
- removed CHARGEOUT1, EXTPOW1, PCBIN: PRT-10474, PRT-10474:PRT-10474
- removed SPCON1: (no value), con-wago-500:W237-102
- removed X4, X5: B4B-ZR, con-jst:B4B-ZR
- added C11, C12, C13, C14: 0.1uF, SparkFun-Capacitors:10NF-0603-50V-10%
- added C15, C16, C17: 10nF, SparkFun-Capacitors:10NF-0603-50V-10%
- added D1: BAS40, diode:BAS40
- added DCIN, DCOUT, MOTOR_L_IN, MOTOR_L_OUT, MOTOR_R_IN, MOTOR_R_OUT, PCBPOWER, PCB_IN, PCB_OUT: PRT-10474, PRT-10474:PRT-10474
- added ESP8266_HEADER: (no value), con-lstb:MA04-2
- added GPS_HEADER, J1: (no value), AMP_MTA:MTA09-100
- added IC4: LTC6811-1, LTC6811-1:LTC6811-1
- added IC5: STM32F407VGT6, STM32F407VGT6:STM32F407VGT6
- added J5, J6: (no value), AMP_MTA:MTA06-100
- added L1: (no value), inductor-neosid:SM-1206
- added LASER_HEADER: (no value), AMP_MTA:MTA10-100
- added LDO_HEADER: (no value), AMP_MTA:MTA02-100
- added LEFT_MOTOR, RIGHT_MOTOR: (no value), AMP_MTA:MTA05-100
- added MOTOR_L_SENSE_IN, MOTOR_L_SENSE_OUT, MOTOR_R_SENSE_IN, MOTOR_R_SENSE_OUT, PCB_SENSE_IN, PCB_SENSE_OUT: JST-XH-04-PIN-LONG-PAD, Rembrandt Electronics - JST XH Connectors v1-0:JST-XH-04-PIN-LONG-PAD
- added Q3, Q4, Q5, Q6, Q7: IRLML5203, transistor-power:IRLML5203
- added Q8: (no value), semicon-smd-ipc:NPN-TRANSISTIOR-2COLSOT89
- added R10, R9: 10K, resistor:R-EU_R0805
- added R11: 15k, resistor:R-EU_R0805
- added R12: 18k, resistor:R-EU_R0805
- added R13: 15K, rcl:R-EU_M0805
- added R14: 18K, rcl:R-EU_M0805
- added R15, R18: 100, rcl:R-EU_M0805
- added R16: 20k, rcl:R-EU_M0805
- added R17: 5k, rcl:R-EU_M0805
- added U5: (no value), adafruit:GPS_FGPMMOPA6H
- added Y1: ASV-25.000MHZ-EJ-T, ASV-25.000MHZ-EJ-T:ASV-25.000MHZ-EJ-T
- C10: value 100nF -> 10uF
- C5: value 22uF -> 100nF
- C9: value 10uF -> 22uF
- IC1: value STM32F407VGT6 -> LD1117S33CTR; device STM32F407VGT6:STM32F407VGT6 -> LD1117S33CTR:LD1117S33CTR
- IC2: value LD1117S33CTR -> MLX90393ELW-ABA-011-SP; device LD1117S33CTR:LD1117S33CTR -> MLX90393ELW-ABA-011-SP:MLX90393ELW-ABA-011-SP
- IC3: value LTC6811-1 -> MLX90393ELW-ABA-011-SP; device LTC6811-1:LTC6811-1 -> MLX90393ELW-ABA-011-SP:MLX90393ELW-ABA-011-SP
- R1: value 51K -> 43k
- R2: value 75K -> 51k
- R5: value 51k -> 75K
- R6: value 43k -> 51K
- X1: value (none) -> Raspi Power Supply
- X2: value (none) -> LTE Model Power Supply
- X6: value B4B-ZR -> Solar Pannel Power; device con-jst:B4B-ZR -> con-wago-500:W237-102
Connections:
- removed net 12V: C1.1, C2.1, C3.1, C7.1, PCBIN.POS, U1.POSITIVE_INPUT, U2.POSITIVE_INPUT, U3.POSITIVE_INPUT, U4.POSITIVE_INPUT
- new net C_GND: C11.1, C12.1, IC3.N/C_1, IC3.N/C_2, IC3.N/C_3, IC3.N/C_4, IC3.N/C_5, IC3.VSS, J6.6, R12.2
- new net C_VDD: C11.2, IC3.VDD, J6.1, R11.1
- new net L_PWM: LEFT_MOTOR.1
- new net MOTOR_R_IN: MOTOR_R_IN.POS, MOTOR_R_OUT.POS
- new net N$1: PCB_SENSE_IN-4.S, PCB_SENSE_OUT-4.S
- new net N$10: Q2.D, R3.1, R5.1, X1.1
- new net N$11: CONVPOW.POS, D1.C, Q1.D
- new net N$12: C7.1, R1.1, R7.1, U2.POSITIVE_OUTPUT, X2.1
- new net N$13: PCB_SENSE_IN-1.S, PCB_SENSE_OUT-1.S
- new net N$14: MOTOR_R_SENSE_IN-4.S, MOTOR_R_SENSE_OUT-4.S
- new net N$16: MOTOR_R_SENSE_IN-3.S, MOTOR_R_SENSE_OUT-3.S
- new net N$17: MOTOR_R_SENSE_IN-2.S, MOTOR_R_SENSE_OUT-2.S
- new net N$18: MOTOR_R_SENSE_IN-1.S, MOTOR_R_SENSE_OUT-1.S
- new net N$19: MOTOR_L_SENSE_IN-4.S, MOTOR_L_SENSE_OUT-4.S
- new net N$20: MOTOR_L_SENSE_IN-3.S, MOTOR_L_SENSE_OUT-3.S
- new net N$21: MOTOR_L_SENSE_IN-2.S, MOTOR_L_SENSE_OUT-2.S
- new net N$22: MOTOR_L_SENSE_IN-1.S, MOTOR_L_SENSE_OUT-1.S
- new net N$23: MOTOR_L_IN.GND, MOTOR_L_OUT.GND
- new net N$24: MOTOR_L_IN.POS, MOTOR_L_OUT.POS
- new net N$25: MOTOR_R_IN.GND, MOTOR_R_OUT.GND
- new net N$27: Q8.C, R18.2
- new net N$28: IC4.V+, PCB_IN.POS, PCB_OUT.POS
- new net N$29: IC3.A0
- new net N$30: IC3.A1
- new net N$31: C12.2, IC3.SENB/CS, IC3.VDD_IO, R10.1, R11.2, R12.1, R9.1
- new net N$32: IC3.INT, J6.5
- new net N$33: IC3.INT/TRIG, J6.2
- new net N$34: IC3.SCL/SCLK, J6.4, R9.2
- new net N$35: IC4.SDO_(NC), R17.2
- new net N$36: IC3.SDA/MOSI, J6.3, R10.2
- new net N$37: IC4.IPB, R15.2
- new net N$38: C14.1, IC2.VDD_IO, R13.1, R14.2
- new net N$39: IC4.IMB, R15.1
- new net N$40: IC4.IBIAS, IC4.ICMP, R16.2
- new net N$42: IC4.SDI_(NC)
- new net N$43: IC4.SCK_(IPA
- new net N$44: IC4.CSB_(IMA)
- new net N$45: C16.1, IC4.VREF1
- new net N$46: C15.1, IC4.VREF2
- new net N$47: C17.1, Q8.E
- new net N$48: IC4.DRIVE, Q8.B
- new net N$8: PCB_SENSE_IN-2.S, PCB_SENSE_OUT-2.S
- new net PCB_GND: C15.2, C16.2, C17.2, IC4.ISOMD, IC4.V-_1, IC4.V-_2, PCB_IN.GND, PCB_OUT.GND, R16.1
- new net R_PWM: RIGHT_MOTOR.5
- new net VBAT: C1.1, C2.1, C3.1, C4.1, PCBPOWER.POS, U1.POSITIVE_INPUT, U2.POSITIVE_INPUT, U3.POSITIVE_INPUT, U4.POSITIVE_INPUT
- net GDC: now also DCIN.GND, DCOUT.GND, X6-1.KL; no longer CHARGEOUT1.GND, EXTPOW1.GND, SPCON1-1.KL
- net GND: now also C13.1, C14.2, CONVPOW.GND, D1.A, IC1.GROUND, IC2.A0, IC2.A1, IC2.N/C_1, IC2.N/C_2, IC2.N/C_3, IC2.N/C_4, IC2.N/C_5, IC2.VSS, J5.6, LASER_HEADER.5, LASER_HEADER.7, LASER_HEADER.9, LEFT_MOTOR.3, PCBPOWER.GND, R14.1, R2.2, R6.2, RIGHT_MOTOR.3, X1.4, X2.4, Y1.GND/CASE; no longer IC2.GROUND, PCBIN.GND, R1.2, R5.2
- net N$2: now also C9.1, Q1.S, U4.POSITIVE_OUTPUT; no longer C4.1, U1.POSITIVE_OUTPUT
- net N$3: now also C6.1, Q2.S, U1.POSITIVE_OUTPUT; no longer C5.1, R2.1, R3.1, U2.POSITIVE_OUTPUT
- net N$4: now also PCB_SENSE_IN-3.S, PCB_SENSE_OUT-3.S; no longer C6.1, R6.1, R7.1, U4.POSITIVE_OUTPUT
- net N$5: now also X6-2.KL; no longer SPCON1-2.KL
- net N$6: now also R5.2, R6.1; no longer R1.1, R2.2
- net N$7: now also R1.2, R2.1; no longer R5.1, R6.2
- net VCC: now also C13.2, C5.1, IC1.VOUT, IC2.VDD, J5.1, R13.2, R17.1, Y1.VDD; no longer C10.1, IC2.VOUT
- net VDC: now also DCIN.POS, DCOUT.POS; no longer CHARGEOUT1.POS, EXTPOW1.POS
- net VDD: now also C10.1, IC1.VIN, LASER_HEADER.10, LASER_HEADER.6, LASER_HEADER.8; no longer C9.1, IC2.VIN
Other:
- note added: "5V Rail"
- note added: "GND INT SCL/SCLK SDA/MOSI INT/TRIG VCC"
- note added: "LTE Modem Power Supply"
- note added: "VCC INT/TRIG SDA/MOSI SCL/SCLK INT GND"
- note removed: "Power Regulation For PCB"

Commit message: updating PCB
Parts:
- removed D1: BAS40, diode:BAS40
- removed IC1: LD1117S33CTR, LD1117S33CTR:LD1117S33CTR
- removed IC4, IC6, IC7: LTC6811-1, LTC6811-1:LTC6811-1
- removed J1: (no value), AMP_MTA:MTA09-100
- removed L1: (no value), inductor-neosid:SM-1206
- added C18: 100nF, resistor:C-EUC1206
- added C19, C20: 0.1uF, resistor:C-EUC0805
- added MOTOR_L_CELL2_DIFF, MOTOR_L_CELL3_DIFF, MOTOR_R_CELL2_DIFF, MOTOR_R_CELL3_DIFF, PCB_CELL2_DIFF, PCB_CELL3_DIFF: INA148UA, INA148UA:INA148UA
- added Q9: IRF512, transistor-power:IRF512
- added R19, R20, R21, R22, R23, R24, R25, R26, R27, R28, R29, R30, R31, R32, R33, R34: 5k, resistor:R-US_R1206
- C1, C2, C3, C4, C6, C7, C8, C9: device SparkFun-Capacitors:10NF-0603-50V-10% -> SparkFun-Capacitors:22UF-0805-6.3V-20%
- C10: device SparkFun-Capacitors:10NF-0603-50V-10% -> SparkFun-Capacitors:10UF-1206-6.3V-20%
- C11, C12, C13, C14: device SparkFun-Capacitors:10NF-0603-50V-10% -> resistor:C-EUC1206
- C15, C16, C17: value 10nF -> 0.1uF; device SparkFun-Capacitors:10NF-0603-50V-10% -> resistor:C-EUC0805
- C5: value 100nF -> 0.1uF; device SparkFun-Capacitors:10NF-0603-50V-10% -> resistor:C-EUC0805
- D2: value (none) -> 1N4446; device eagle-ltspice:DIODE_E- -> diode:1N4446
- Q1, Q2, Q3, Q4, Q5, Q6, Q7: value IRLML5203 -> IRF512; device transistor-power:IRLML5203 -> transistor-power:IRF512
- Q8: value (none) -> IRF512; device semicon-smd-ipc:NPN-TRANSISTIOR-2COLSOT89 -> transistor-power:IRF512
- R1, R2, R3, R4, R5, R6, R7, R8: device resistor:R-EU_R0805 -> resistor:R-EU_R1206
- R15: value 100 -> 2.2k; device rcl:R-EU_M0805 -> resistor:R-EU_R1206
- R16: value 20k -> 2.2k; device rcl:R-EU_M0805 -> resistor:R-EU_R1206
- R17: device rcl:R-EU_M0805 -> resistor:R-US_R1206
- R18: value 100 -> 5k; device rcl:R-EU_M0805 -> resistor:R-US_R1206
- U5: value (none) -> AMS1117-3.3; device adafruit:GPS_FGPMMOPA6H -> AMS1117-3.3:AMS1117-3.3
Connections:
- removed net MOTOR_R_IN: MOTOR_R_IN.POS, MOTOR_R_OUT.POS
- removed net N$18: MOTOR_R_SENSE_IN-1.S, MOTOR_R_SENSE_OUT-1.S
- removed net N$21: MOTOR_L_SENSE_IN-2.S, MOTOR_L_SENSE_OUT-2.S
- removed net N$22: MOTOR_L_SENSE_IN-1.S, MOTOR_L_SENSE_OUT-1.S
- removed net N$23: MOTOR_L_IN.GND, MOTOR_L_OUT.GND
- removed net N$24: MOTOR_L_IN.POS, MOTOR_L_OUT.POS
- removed net N$25: MOTOR_R_IN.GND, MOTOR_R_OUT.GND
- removed net N$40 (its old number): IC4.IBIAS, IC4.ICMP, R16.2
- removed net N$44: IC4.CSB_(IMA)
- removed net N$46 (its old number): C15.1, IC4.VREF2
- removed net PCB_GND: C15.2, C16.2, C17.2, IC4.ISOMD, IC4.V-_1, IC4.V-_2, PCB_IN.GND, PCB_OUT.GND, R16.1
- new net N$1: PCB_CELL2_DIFF.+IN, PCB_SENSE_IN-3.S, PCB_SENSE_OUT-3.S
- new net N$14: MOTOR_L_CELL3_DIFF.-IN, MOTOR_L_SENSE_IN-1.S, MOTOR_L_SENSE_OUT-1.S, R32.1
- new net N$19: R33.2
- new net N$41: C15.2, C17.2, PCB_CELL2_DIFF.REF, PCB_CELL2_DIFF.V-, PCB_CELL3_DIFF.REF, PCB_CELL3_DIFF.V-, PCB_IN.GND, PCB_OUT.GND, R20.1, R29.2
- new net N$49: R21.1, R22.2
- new net N$50: C16.2, C5.2, MOTOR_L_CELL2_DIFF.REF, MOTOR_L_CELL2_DIFF.V-, MOTOR_L_CELL3_DIFF.REF, MOTOR_L_CELL3_DIFF.V-, MOTOR_L_IN.GND, MOTOR_L_OUT.GND, R24.1
- new net N$51: MOTOR_L_CELL2_DIFF.OUT, R23.2
- new net N$52: R23.1, R24.2
- new net N$53: MOTOR_R_CELL2_DIFF.+IN, MOTOR_R_SENSE_IN-3.S, MOTOR_R_SENSE_OUT-3.S
- new net N$54: MOTOR_R_CELL3_DIFF.-IN, MOTOR_R_SENSE_IN-1.S, MOTOR_R_SENSE_OUT-1.S, R34.1
- new net N$55: MOTOR_R_CELL2_DIFF.-IN, MOTOR_R_CELL3_DIFF.+IN, MOTOR_R_SENSE_IN-2.S, MOTOR_R_SENSE_OUT-2.S
- new net N$57: C19.1, C20.1, MOTOR_R_CELL2_DIFF.V+, MOTOR_R_CELL3_DIFF.V+, MOTOR_R_IN.POS, MOTOR_R_OUT.POS, R26.1
- new net N$58: MOTOR_R_CELL3_DIFF.OUT, R25.2
- new net N$59: R25.1, R26.2
- new net N$60: C19.2, C20.2, MOTOR_R_CELL2_DIFF.REF, MOTOR_R_CELL2_DIFF.V-, MOTOR_R_CELL3_DIFF.REF, MOTOR_R_CELL3_DIFF.V-, MOTOR_R_IN.GND, MOTOR_R_OUT.GND, R28.1
- new net N$61: MOTOR_R_CELL2_DIFF.OUT, R27.2
- new net N$62: R27.1, R28.2
- new net PCB_IN: C15.1, C17.1, PCB_CELL2_DIFF.V+, PCB_CELL3_DIFF.V+, PCB_IN.POS, PCB_OUT.POS, R18.1
- net GND: now also C18.2, Q1.D, Q8.D, R15.1, R16.1; no longer C5.2, CONVPOW.GND, D1.A, IC1.GROUND, R4.2, R6.2, X1.4
- net N$10: now also Q1.G, R16.2; no longer Q2.D, R3.1, R5.1, X1.1
- net N$11: now also CONVPOW.GND, Q8.S; no longer CONVPOW.POS, D1.C, Q1.D
- net N$13: now also R29.1, R30.2; no longer PCB_SENSE_IN-1.S, PCB_SENSE_OUT-1.S
- net N$16: now also R31.2; no longer MOTOR_R_SENSE_IN-3.S, MOTOR_R_SENSE_OUT-3.S
- net N$17: now also R31.1, R32.2; no longer MOTOR_R_SENSE_IN-2.S, MOTOR_R_SENSE_OUT-2.S
- net N$2: now also CONVPOW.POS; no longer Q1.S
- net N$20: now also R33.1, R34.2; no longer MOTOR_L_SENSE_IN-3.S, MOTOR_L_SENSE_OUT-3.S
- net N$27: now also PCB_CELL2_DIFF.-IN, PCB_CELL3_DIFF.+IN, PCB_SENSE_IN-2.S, PCB_SENSE_OUT-2.S; no longer Q8.C, R18.2
- net N$28: now also Q8.G, R15.2; no longer IC4.V+, PCB_IN.POS, PCB_OUT.POS
- net N$3: now also R3.1, R5.1, X1.1; no longer Q2.S
- net N$35: now also Q1.S, R4.2, R6.2, X1.4; no longer IC4.SDO_(NC), R17.2
- net N$37: now also R17.1, R18.2; no longer IC4.IPB, R15.2
- net N$39: now also PCB_CELL2_DIFF.OUT, R19.2; no longer IC4.IMB, R15.1
- net N$4: now also PCB_CELL3_DIFF.OUT, R17.2; no longer PCB_SENSE_IN-3.S, PCB_SENSE_OUT-3.S
- net N$42: now also R19.1, R20.2; no longer IC4.SDI_(NC)
- net N$43: now also MOTOR_L_CELL2_DIFF.+IN, MOTOR_L_SENSE_IN-3.S, MOTOR_L_SENSE_OUT-3.S; no longer IC4.SCK_(IPA
- net N$45: now also MOTOR_L_CELL2_DIFF.-IN, MOTOR_L_CELL3_DIFF.+IN, MOTOR_L_SENSE_IN-2.S, MOTOR_L_SENSE_OUT-2.S; no longer C16.1, IC4.VREF1
- net N$47: now also C16.1, C5.1, MOTOR_L_CELL2_DIFF.V+, MOTOR_L_CELL3_DIFF.V+, MOTOR_L_IN.POS, MOTOR_L_OUT.POS, R22.1; no longer C17.1, Q8.E
- net N$48: now also MOTOR_L_CELL3_DIFF.OUT, R21.2; no longer IC4.DRIVE, Q8.B
- net N$5: now also D2.A; no longer D2.C
- net N$8: now also PCB_CELL3_DIFF.-IN, PCB_SENSE_IN-1.S, PCB_SENSE_OUT-1.S, R30.1; no longer PCB_SENSE_IN-2.S, PCB_SENSE_OUT-2.S
- net VCC: now also C18.1, U5.VOUT; no longer C5.1, IC1.VOUT, R17.1
- net VDC: now also D2.C; no longer D2.A
- net VDD: no longer IC1.VIN
