File: PCB.sch (EAGLE design)
At the start: 153 parts, among them IC3 MLX90393ELW-ABA-011-SP, IC5 STM32F407VGT6, Q10 2N3906, Q11 8Mhz, Q12 2N3906, Q13 2N3906, Q14 2N3906, Q15 2N3906

Commit message: update
Parts:
- GPS_HEADER: device AMP_MTA:MTA09-100 -> con-amp:MTA04-100
Connections:
- removed net CMP_CS: SPI_CMP.SENB/CS
- removed net ESP_EN: ESP8266_HEADER.4
- removed net N$10: R16.2, RASPI_SW.G
- removed net N$13: R29.1, R30.2
- removed net N$17: R31.1, R32.2
- removed net N$19: Q15.C, R47.2
- removed net N$20: R33.1, R34.2
- removed net N$28: CON_SW.G, R15.2
- removed net N$37: R17.1, R18.2
- removed net N$42: R19.1, R20.2
- removed net N$49: R21.1, R22.2
- removed net N$52: R23.1, R24.2
- removed net N$59: R25.1, R26.2
- removed net N$62: R27.1, R28.2
- removed net N$75: Q10.C, R39.2
- removed net N$78: Q12.C, R41.2
- removed net N$80: Q13.C, R43.2
- removed net N$82: Q14.C, R45.2
- new net C_MOS: CON_SW.G, IC5.PA10, R15.2
- new net GPS_RX: GPS_HEADER.2, IC5.PB6
- new net GPS_TX: GPS_HEADER.3, IC5.PB7
- new net LASER_MOS: IC5.PA12, LASR_SW.G
- new net LDR0: IC5.PA0, Q10.C, R39.2
- new net LDR1: IC5.PA1, Q12.C, R41.2
- new net LDR2: IC5.PA2, Q13.C, R43.2
- new net LDR3: IC5.PA3, Q15.C, R47.2
- new net LDR4: IC5.PA4, Q14.C, R45.2
- new net LDR_MOS: IC5.PA15, LDR_SW.G
- new net L_MOS: IC5.PA8, LM_SW.G
- new net MOTOR_L_CELL1: IC5.PB0, R31.1, R32.2
- new net MOTOR_L_CELL2: IC5.PB1, R23.1, R24.2
- new net MOTOR_L_CELL3: IC5.PC0, R21.1, R22.2
- new net MOTOR_R_CELL1: IC5.PC1, R33.1, R34.2
- new net MOTOR_R_CELL2: IC5.PC2, R27.1, R28.2
- new net MOTOR_R_CELL3: IC5.PC3, R25.1, R26.2
- new net PCB_CELL1: IC5.PA5, R29.1, R30.2
- new net PCB_CELL2: IC5.PA6, R19.1, R20.2
- new net PCB_CELL3: IC5.PA7, R17.1, R18.2
- new net RASPI_MOS: IC5.PA11, R16.2, RASPI_SW.G
- new net R_MOS: IC5.PA9, RM_SW.G
- net CMP_INT: now also IC5.PE9
- net CMP_MISO: now also IC5.PB14
- net CMP_MOSI: now also IC5.PB15
- net CMP_SCL: now also IC5.PB8
- net CMP_SCLK: now also IC5.PB13
- net CMP_SDA: now also IC5.PB9
- net CMP_SPI_INT: now also IC5.PE7
- net CMP_TRG: now also IC5.PE10
- net CMP_TRIG: now also IC5.PE8
- net ESP_RX: now also IC5.PB10; no longer IC5.PA9
- net ESP_TX: now also IC5.PB11; no longer IC5.PA10
- net GND: now also GPS_HEADER.4, SPI_CMP.SENB/CS
- net L_PWM: now also IC5.PC6
- net R_PWM: now also IC5.PC7
- net VCC: now also ESP8266_HEADER.4, GPS_HEADER.1
Other:
- moved on the sheet: JP3, LDR_SW, R13, R14, R37, R39, R40, R41, R42, R43, R44, R45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

Commit message: update
Parts:
- removed C15, C16, C17, C19, C20, C5: 0.1uF, rcl:C-EUC1206
- removed MOTOR_L_CELL2, MOTOR_L_CELL3, MOTOR_R_CELL2, MOTOR_R_CELL3, PCB_CELL2, PCB_CELL3: INA148UA, INA148UA:INA148UA
- removed R17, R18, R19, R20, R21, R22, R23, R24, R25, R26, R27, R28, R29, R30, R31, R32, R33, R34: 5k, resistor:R-US_R1206
- added C23: 100uF, rcl:C-EUC1206
- LTE_PWR: value LTE Model Power Supply -> LTE Modem Power Supply; device con-berg:PN87520 -> MOLEX_USB:105057-0001
- PWR: value PWR -> RED
- R15, R16: value 2.2k -> 10k
- RASPI_PWR: device con-berg:PN87520 -> MOLEX_USB:105057-0001
- RST: value RST -> RED
Connections:
- removed net N$35: R4.2, R6.2, RASPI_PWR.4, RASPI_SW.S
- removed net N$39: PCB_CELL2.OUT, R19.2
- removed net N$4: PCB_CELL3.OUT, R17.2
- removed net N$48: MOTOR_L_CELL3.OUT, R21.2
- removed net N$51: MOTOR_L_CELL2.OUT, R23.2
- removed net N$58: MOTOR_R_CELL3.OUT, R25.2
- removed net N$61: MOTOR_R_CELL2.OUT, R27.2
- new net N$19: RASPI_SW.S, RASPI_SW_REG.COMMON(GROUND)
- net GND: now also C23.2, CONVPOW.GND, R4.2, R6.2, RASPI_PWR.4; no longer CONV_SW_REG.COMMON(GROUND), MICRO_REG.ADJ/GND, RASPI_SW_REG.COMMON(GROUND)
- net MOTOR_L_CELL1: no longer R31.1, R32.2
- net MOTOR_L_CELL2: no longer R23.1, R24.2
- net MOTOR_L_CELL3: no longer R21.1, R22.2
- net MOTOR_R_CELL1: no longer R33.1, R34.2
- net MOTOR_R_CELL2: no longer R27.1, R28.2
- net MOTOR_R_CELL3: no longer R25.1, R26.2
- net N$1: no longer PCB_CELL2.+IN
- net N$11: now also CONV_SW_REG.COMMON(GROUND); no longer CONVPOW.GND
- net N$14: no longer MOTOR_L_CELL3.-IN, R32.1
- net N$27: no longer PCB_CELL2.-IN, PCB_CELL3.+IN
- net N$41: no longer C15.2, C17.2, PCB_CELL2.REF, PCB_CELL2.V-, PCB_CELL3.REF, PCB_CELL3.V-, R18.1, R20.1, R29.2
- net N$43: no longer MOTOR_L_CELL2.+IN
- net N$45: no longer MOTOR_L_CELL2.-IN, MOTOR_L_CELL3.+IN
- net N$47: no longer C16.1, C5.1, MOTOR_L_CELL2.V+, MOTOR_L_CELL3.V+
- net N$50: no longer C16.2, C5.2, MOTOR_L_CELL2.REF, MOTOR_L_CELL2.V-, MOTOR_L_CELL3.REF, MOTOR_L_CELL3.V-, R22.1, R24.1, R31.2
- net N$53: no longer MOTOR_R_CELL2.+IN
- net N$54: no longer MOTOR_R_CELL3.-IN, R34.1
- net N$55: no longer MOTOR_R_CELL2.-IN, MOTOR_R_CELL3.+IN
- net N$57: no longer C19.1, C20.1, MOTOR_R_CELL2.V+, MOTOR_R_CELL3.V+
- net N$60: no longer C19.2, C20.2, MOTOR_R_CELL2.REF, MOTOR_R_CELL2.V-, MOTOR_R_CELL3.REF, MOTOR_R_CELL3.V-, R26.1, R28.1, R33.2
- net N$8: no longer PCB_CELL3.-IN, R30.1
- net PCB_CELL1: no longer R29.1, R30.2
- net PCB_CELL2: no longer R19.1, R20.2
- net PCB_CELL3: no longer R17.1, R18.2
- net PCB_IN: no longer C15.1, C17.1, PCB_CELL2.V+, PCB_CELL3.V+
- net VBAT: now also C23.1
Other:
- note removed: "LTE Modem Power Supply"
- moved on the sheet: C1, C10, C18, C2, C3, C4, C6, C7, C8, C9, CONVPOW, CONV_SW_REG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

Commit message: trying to finalize verion 1 of PCB
Parts:
- removed C23: 100uF, rcl:C-EUC1206
- removed C4, C6, C7, C8, C9: 22uF, rcl:C-EUC1206
- removed D2: 1N4446, diode:1N4446
- removed GND, VDD: TEST-POINT3X4, SparkFun-Connectors:TEST-POINT3X4
- removed MOTOR_L_IN, MOTOR_L_OUT, MOTOR_R_IN, MOTOR_R_OUT, PCB_IN, PCB_OUT: PRT-10474, PRT-10474:PRT-10474
- removed MOTOR_R_SENSE_IN: JST-XH-04-PIN-LONG-PAD, Rembrandt Electronics - JST XH Connectors v1-0:JST-XH-04-PIN-LONG-PAD
- removed Q10, Q12, Q13, Q14, Q15: 2N3906, transistor-pnp:2N3906
- added D1, D3: V60D45C-M3_I, V60D45C-M3_I:V60D45C-M3_I
- added ESP_DEBUG: (no value), con-lstb:MA08-1
- added GPS_DEBUG: (no value), con-lstb:MA06-1
- added JP4, JP5: (no value), jumper:JP2E
- added LDR0, LDR1, LDR2, LDR3, LDR4, MOTOR_L_CELL1, MOTOR_L_CELL2, MOTOR_R_CELL1, MOTOR_R_CELL2, PCB_CELL1, PCB_CELL2: TPSQB2,54, testpad:TPSQB2,54
- added LED1: BLUE, led:LEDCHIPLED_0805
- added MOTOR_L_CELL3, MOTOR_R_CELL3, PCB_CELL3: PCB_CELL3, testpad:TPSQB2,54
- added MOTOR_R_SENSE: MOTOR_R_SENSE_IN, bt_con-jst-xh:04-JST-B4B-XH-A
- added PCB_SW: PRT-10474, PRT-10474:PRT-10474
- added R17, R23, R29: 180k, resistor:R-US_R0805
- added R18, R24, R30: 6.2k, resistor:R-US_R0805
- added R19, R25, R31: 8.2k, resistor:R-US_R0805
- added R20, R26, R32: 5.1k, resistor:R-US_R0805
- added R21, R27, R33: 680, resistor:R-US_R0805
- added R22, R28, R34: 2.4k, resistor:R-US_R0805
- added R48: 200, rcl:R-US_R0805
- added R49: 10K, rcl:R-US_R0805
- added R50, R52: 100K, rcl:R-US_R0805
- added R51: 510, rcl:R-US_R0805
- added R53, R54, R55: 100k, resistor:R-US_R1206
- C1, C2, C3: value 22uF -> 100uF; device rcl:C-EUC1206 -> rcl:CPOL-US140CLH-0810
- C10: device rcl:C-EUC1206 -> resistor:C-EUC0805
- C18: value 100nF -> 22uF; device resistor:C-EUC1206 -> resistor:C-EUC0805
- C25, C26, C30, C31, C32, C33, C34, C35, C36, C37, C38, C39, C40, C41, C42, C43, C44, C45: device SparkFun-Capacitors:10UF-1206-6.3V-20% -> resistor:C-EUC0805K
- MOTOR_L_SENSE_IN: value JST-XH-04-PIN-LONG-PAD -> MOTOR_L_SENSE_IN; device Rembrandt Electronics - JST XH Connectors v1-0:JST-XH-04-PIN-LONG-PAD -> bt_con-jst-xh:04-JST-B4B-XH-A
- MOTOR_L_SENSE_OUT, MOTOR_R_SENSE_OUT: value JST-XH-04-PIN-LONG-PAD -> MOTOR_R_SENSE_OUT; device Rembrandt Electronics - JST XH Connectors v1-0:JST-XH-04-PIN-LONG-PAD -> bt_con-jst-xh:04-JST-B4B-XH-A
- PCB_SENSE_IN: value JST-XH-04-PIN-LONG-PAD -> PCB_SENSE_IN; device Rembrandt Electronics - JST XH Connectors v1-0:JST-XH-04-PIN-LONG-PAD -> bt_con-jst-xh:04-JST-B4B-XH-A
- PCB_SENSE_OUT: value JST-XH-04-PIN-LONG-PAD -> PCB_SENSE_OUT; device Rembrandt Electronics - JST XH Connectors v1-0:JST-XH-04-PIN-LONG-PAD -> bt_con-jst-xh:04-JST-B4B-XH-A
- R1, R16, R2, R3, R4, R5, R6, R7, R8: device resistor:R-EU_R1206 -> resistor:R-US_R0805
- R10, R9: device resistor:R-EU_R0805 -> resistor:R-US_R1206
- R11, R12, R13, R14, R35, R36, R38: device resistor:R-EU_R1206 -> rcl:R-US_R0805
- R15: value 10k -> 100k; device resistor:R-EU_R1206 -> resistor:R-US_R0805
- R37, R40, R42, R46: value 2k -> 100k; device rcl:R-EU_R1206 -> resistor:R-US_R1206
- R39, R41: value 1k -> 100k; device rcl:R-EU_R1206 -> resistor:R-US_R1206
- R43: value 1k -> 1M; device rcl:R-EU_R1206 -> resistor:R-US_R0805
- R44: value 2k -> 1M; device rcl:R-EU_R1206 -> resistor:R-US_R0805
- R45: value 1k -> 200; device rcl:R-EU_R1206 -> rcl:R-US_R0805
- R47: value 1k -> 10K; device rcl:R-EU_R1206 -> rcl:R-US_R0805
Connections:
- removed net GDC: DCIN.GND, DCOUT.GND, SOLAR.GND
- removed net N$40: PCB_SENSE_IN-4.S, PCB_SENSE_OUT-4.S
- removed net N$41: PCB_IN.GND, PCB_OUT.GND
- removed net N$53: MOTOR_R_SENSE_IN-3.S, MOTOR_R_SENSE_OUT-3.S
- removed net N$54: MOTOR_R_SENSE_IN-1.S, MOTOR_R_SENSE_OUT-1.S
- removed net N$55: MOTOR_R_SENSE_IN-2.S, MOTOR_R_SENSE_OUT-2.S
- removed net N$56: MOTOR_R_SENSE_IN-4.S, MOTOR_R_SENSE_OUT-4.S
- removed net N$57: MOTOR_R_IN.POS, MOTOR_R_OUT.POS
- removed net N$60: MOTOR_R_IN.GND, MOTOR_R_OUT.GND
- removed net N$64: BOOT0.S, R36.2
- removed net N$74: LDR_HEADER.2, Q10.B, R37.2
- removed net N$76: LDR_HEADER.8, Q15.B, R46.2
- removed net N$77: LDR_HEADER.4, Q12.B, R40.2
- removed net N$79: LDR_HEADER.6, Q13.B, R42.2
- removed net N$85: LDR_HEADER.10, Q14.B, R44.2
- removed net PCB_IN: PCB_IN.POS, PCB_OUT.POS
- removed net VDC: D2.C, DCIN.POS, DCOUT.POS
- new net N$10: MOTOR_L_SENSE_IN-3.1, MOTOR_L_SENSE_OUT-3.1, R27.1
- new net N$12: MOTOR_L_SENSE_IN-2.1, MOTOR_L_SENSE_OUT-2.1, R25.1
- new net N$17: MOTOR_R_SENSE-3.1, MOTOR_R_SENSE_OUT-3.1, R33.1
- new net N$20: MOTOR_R_SENSE-2.1, MOTOR_R_SENSE_OUT-2.1, R31.1
- new net N$28: MOTOR_R_SENSE-1.1, MOTOR_R_SENSE_OUT-1.1, R29.1
- new net N$35: D1.CATHODE_(HEATSINK), D3.CATHODE_(HEATSINK), DCOUT.POS
- new net N$4: D1.ANODE_1, D1.ANODE_2, DCIN.POS
- new net N$48: ESP8266_HEADER.4, ESP8266_HEADER.8, JP4.2
- new net N$49: GPS_HEADER.1, JP5.3
- new net N$51: LASER_HEADER.1, LASER_HEADER.3, LASER_HEADER.5, LASER_HEADER.7, LASER_HEADER.9, LASR_SW.D
- new net N$52: PCBPOWER.POS, PCB_SW.GND
- net CMP_SCL: now also R47.1
- net CMP_SDA: now also R49.1
- net ESP_GPIO0: now also ESP_DEBUG.8
- net ESP_GPIO2: now also ESP_DEBUG.7, R50.1
- net ESP_RX: now also ESP_DEBUG.4
- net ESP_TX: now also ESP_DEBUG.5
- net GND: now also C1.-, C2.-, C3.-, C45.2, DCIN.GND, DCOUT.GND, ESP_DEBUG.1, GPS_DEBUG.1, LED1.C, MICRO_REG.ADJ/GND, MOTOR_L_SENSE_IN-4.1, MOTOR_L_SENSE_OUT-4.1, MOTOR_R_SENSE-4.1, MOTOR_R_SENSE_OUT-4.1, PCB_SENSE_IN-4.1, PCB_SENSE_OUT-4.1, R18.2, R20.2, R22.2, R24.2, R26.2, R28.2, R30.2, R32.2, R34.2, R51.2, RASPI_SW.S, SOLAR.GND; no longer C1.2, C2.2, C23.2, C3.2, C4.2, C45.1, C6.2, C7.2, C8.2, C9.2, GND.1, LASER_HEADER.1, LASER_HEADER.3, LASER_HEADER.5, LASER_HEADER.7, LASER_HEADER.9, R15.1, R37.1, R39.1, R40.1, R41.1, R42.1, R43.1, R44.1, R45.1, R46.1, R47.1, RASPI_SW.D
- net GPS_RX: now also GPS_DEBUG.4
- net GPS_TX: now also GPS_DEBUG.5
- net LASER_MOS: now also R55.1
- net LDR0: now also LDR0.TP, LDR_HEADER.2, R37.1; no longer Q10.C, R39.2
- net LDR1: now also LDR1.TP, LDR_HEADER.4, R39.1; no longer Q12.C, R41.2
- net LDR2: now also LDR2.TP, LDR_HEADER.6, R40.1; no longer Q13.C, R43.2
- net LDR3: now also LDR3.TP, LDR_HEADER.8, R41.1; no longer Q15.C, R47.2
- net LDR4: now also LDR4.TP, LDR_HEADER.10, R42.1; no longer Q14.C, R45.2
- net LDR_MOS: now also R54.1
- net L_MOS: now also R46.2
- net MOTOR_L_CELL1: now also MOTOR_L_CELL1.TP, R27.2, R28.1
- net MOTOR_L_CELL2: now also MOTOR_L_CELL2.TP, R25.2, R26.1
- net MOTOR_L_CELL3: now also MOTOR_L_CELL3.TP, R23.2, R24.1
- net MOTOR_R_CELL1: now also MOTOR_R_CELL1.TP, R33.2, R34.1
- net MOTOR_R_CELL2: now also MOTOR_R_CELL2.TP, R31.2, R32.1
- net MOTOR_R_CELL3: now also MOTOR_R_CELL3.TP, R29.2, R30.1
- net N$1: now also PCB_SENSE_IN-3.1, PCB_SENSE_OUT-3.1, R21.1; no longer PCB_SENSE_IN-3.S, PCB_SENSE_OUT-3.S
- net N$11: now also R43.2
- net N$14: now also MOTOR_L_SENSE_IN-1.1, MOTOR_L_SENSE_OUT-1.1, R23.1; no longer MOTOR_L_SENSE_IN-1.S, MOTOR_L_SENSE_OUT-1.S
- net N$16: now also C2.+; no longer C6.1
- net N$19: now also R44.2, RASPI_SW.D; no longer RASPI_SW.S
- net N$2: no longer C9.1
- net N$27: now also PCB_SENSE_IN-2.1, PCB_SENSE_OUT-2.1, R19.1; no longer PCB_SENSE_IN-2.S, PCB_SENSE_OUT-2.S
- net N$43: now also IC5.PD15, R45.1; no longer MOTOR_L_SENSE_IN-3.S, MOTOR_L_SENSE_OUT-3.S
- net N$44: now also R52.2
- net N$45: now also BOOT0.S, R51.1; no longer MOTOR_L_SENSE_IN-2.S, MOTOR_L_SENSE_OUT-2.S
- net N$46: now also GPS_DEBUG.3, JP5.1; no longer MOTOR_L_SENSE_IN-4.S, MOTOR_L_SENSE_OUT-4.S
- net N$47: now also LDR_SW.D, R37.2, R39.2, R40.2, R41.2, R42.2; no longer MOTOR_L_IN.POS, MOTOR_L_OUT.POS
- net N$5: now also D3.ANODE_1, D3.ANODE_2; no longer D2.A
- net N$50: now also LED1.A, R45.2; no longer MOTOR_L_IN.GND, MOTOR_L_OUT.GND
- net N$6: now also C1.+; no longer C7.1
- net N$69: now also BOOT0.D
- net N$71: now also R46.1
- net N$72: now also R53.1
- net N$8: now also PCB_SENSE_IN-1.1, PCB_SENSE_OUT-1.1, R17.1; no longer PCB_SENSE_IN-1.S, PCB_SENSE_OUT-1.S
- net N$9: no longer LTE_PWR.2
- net PCB_CELL1: now also PCB_CELL1.TP, R21.2, R22.1
- net PCB_CELL2: now also PCB_CELL2.TP, R19.2, R20.1
- net PCB_CELL3: now also PCB_CELL3.TP, R17.2, R18.1
- net R_MOS: now also R53.2
- net VBAT: now also PCB_SW.POS, R15.1, R43.1, R44.1; no longer C1.1, C2.1, C23.1, C3.1, C4.1, PCBPOWER.POS
- net VCC: now also C45.1, ESP_DEBUG.3, JP4.1, JP4.3, JP5.2, R36.2, R47.2, R48.1, R48.2, R49.2, R50.2, R52.1, R54.2, R55.2; no longer BOOT0.D, C45.2, ESP8266_HEADER.4, ESP8266_HEADER.8, GPS_HEADER.1, VDD.1
- net VDD: now also C3.+; no longer C8.1, LASR_SW.D, LDR_SW.D, Q10.E, Q12.E, Q13.E, Q14.E, Q15.E
Other:
- note removed: "For Each VDD"
- moved on the sheet: BOOT0, C10, C26, C38, C45, CONV_SW_REG, CON_SW, DCIN, DCOUT, GPS_HEADER, JP2, JP3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

Commit message: update
Parts:
- removed C24: 100nF, SparkFun-Capacitors:10UF-1206-6.3V-20%
- removed C36, C37: 100nF, resistor:C-EUC0805K
- added C4: 100uF, rcl:CPOL-US140CLH-0810
- added C5: 100nF, rcl:C-EUC0805
- added R56: 200, rcl:R-US_R0805
- BOOT0, NRST: value (none) -> IRF512; device zetex:NMOSSOT23 -> transistor-power:IRF512
- C25, C26, C30, C32, C33, C34, C38, C39, C40, C41, C42, C43, C44, C45: device resistor:C-EUC0805K -> rcl:C-EUC0805
- C31: value 1uF -> 100nF; device resistor:C-EUC0805K -> rcl:C-EUC0805
- C35: value 100nF -> 1uF; device resistor:C-EUC0805K -> rcl:C-EUC0805
- renumbered MOTOR_L_CELL1 to L_CELL1, MOTOR_L_CELL2 to L_CELL2, MOTOR_L_CELL3 to L_CELL3, MOTOR_R_CELL1 to R_CELL1, MOTOR_R_CELL2 to R_CELL2, MOTOR_R_CELL3 to R_CELL3, MOTOR_R_SENSE to MOTOR_R_SENSE_IN, PCB_CELL1 to PCB1, PCB_CELL2 to PCB2, PCB_CELL3 to PCB3
Connections:
- removed net ESP_RST: ESP8266_HEADER.6
- removed net N$180: C30.1, C35.1, IC5.VDDA, IC5.VREF+, R11.1
- new net N$37: PWR.A, R48.2
- new net N$39: C30.1, C35.1, IC5.VREF+, R11.1
- new net N$40: C31.1, C34.1, IC5.VDDA, L1.1, R11.2
- new net N$41: ESP_DEBUG.3, JP4.3
- net GND: now also C31.2, C34.2, C4.-, C5.2, CON_SW.S, R15.1; no longer C24.1, C31.1, C34.1, C36.2, C37.2, CON_SW.D, R16.1
- net N$11: now also CON_SW.D; no longer CON_SW.S
- net N$34: now also R56.1, RST.A; no longer C31.2, C34.2, C36.1, C37.1, L1.1, R11.2
- net N$63: now also C5.1, R56.2; no longer C24.2, RST.A
- net N$9: now also LTE_PWR.2
- net VBAT: now also R16.1; no longer R15.1
- net VCC: now also C4.+; no longer ESP_DEBUG.3, JP4.3, PWR.A, R48.2
Other:
- moved on the sheet: C30, C31, C34, C35, L1, R11, R15, R16, R52, RST

Commit message: revised
Connections:
- removed net N$18: C11.1, CMP_BRKOUT.1, IC3.A0, IC3.A1, IC3.VDD
- removed net N$31: CMP_BRKOUT.5, IC3.N/C_3
- removed net N$32: C12.2, CMP_BRKOUT.7, IC3.N/C_2
- removed net N$33: C21.1, CMP_BRKOUT.9, IC3.N/C_1
- net N$21: now also C12.2, C21.1, CMP_BRKOUT.5, CMP_BRKOUT.7, CMP_BRKOUT.9, IC3.N/C_1, IC3.N/C_2, IC3.N/C_3
- net N$30: now also C11.1, CMP_BRKOUT.1, IC3.A0, IC3.A1, IC3.VDD
Changed lines of the file:
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@@
 </busses>
 <nets>
-<net name="N$18" class="0">
-<segment>
-<pinref part="CMP_BRKOUT" gate="G$1" pin="1"/>
-<wire x1="76.2" y1="124.46" x2="76.2" y2="157.48" width="0.1524" layer="91"/>
-<wire x1="76.2" y1="157.48" x2="139.7" y2="157.48" width="0.1524" layer="91"/>
-<pinref part="IC3" gate="G$1" pin="VDD"/>
-<wire x1="139.7" y1="157.48" x2="139.7" y2="147.32" width="0.1524" layer="91"/>
-<pinref part="C11" gate="G$1" pin="1"/>
-<wire x1="139.7" y1="157.48" x2="144.78" y2="157.48" width="0.1524" layer="91"/>
-<junction x="139.7" y="157.48"/>
-<wire x1="144.78" y1="157.48" x2="157.48" y2="157.48" width="0.1524" layer="91"/>
-<junction x="144.78" y="157.48"/>
-<pinref part="IC3" gate="G$1" pin="A1"/>
-<wire x1="157.48" y1="119.38" x2="162.56" y2="119.38" width="0.1524" layer="91"/>
-<wire x1="162.56" y1="119.38" x2="162.56" y2="121.92" width="0.1524" layer="91"/>
-<wire x1="162.56" y1="121.92" x2="162.56" y2="157.48" width="0.1524" layer="91"/>
-<wire x1="162.56" y1="157.48" x2="157.48" y2="157.48" width="0.1524" layer="91"/>
-<pinref part="IC3" gate="G$1" pin="A0"/>
-<wire x1="157.48" y1="121.92" x2="162.56" y2="121.92" width="0.1524" layer="91"/>
-<junction x="162.56" y="121.92"/>
-</segment>
-</net>
 <net name="N$21" class="0">
 <segment>
@@
 <wire x1="101.6" y1="149.86" x2="101.6" y2="132.08" width="0.1524" layer="91"/>
 <junction x="101.6" y="132.08"/>
+<pinref part="CMP_BRKOUT" gate="G$1" pin="5"/>
+<wire x1="76.2" y1="119.38" x2="66.04" y2="119.38" width="0.1524" layer="91"/>
+<wire x1="66.04" y1="119.38" x2="66.04" y2="83.82" width="0.1524" layer="91"/>
+<wire x1="66.04" y1="83.82" x2="66.04" y2="66.04" width="0.1524" layer="91"/>
+<wire x1="66.04" y1="66.04" x2="162.56" y2="66.04" width="0.1524" layer="91"/>
+<pinref part="IC3" gate="G$1" pin="N/C_3"/>
+<wire x1="162.56" y1="66.04" x2="162.56" y2="116.84" width="0.1524" layer="91"/>
+<wire x1="162.56" y1="116.84" x2="157.48" y2="116.84" width="0.1524" layer="91"/>
+<wire x1="76.2" y1="121.92" x2="76.2" y2="119.38" width="0.1524" layer="91"/>
+<junction x="76.2" y="121.92"/>
+<junction x="76.2" y="119.38"/>
+<pinref part="CMP_BRKOUT" gate="G$1" pin="7"/>
+<wire x1="76.2" y1="116.84" x2="68.58" y2="116.84" width="0.1524" layer="91"/>
+<wire x1="68.58" y1="116.84" x2="68.58" y2="83.82" width="0.1524" layer="91"/>
+<wire x1="68.58" y1="83.82" x2="68.58" y2="68.58" width="0.1524" layer="91"/>
+<wire x1="68.58" y1="68.58" x2="142.24" y2="68.58" width="0.1524" layer="91"/>
+<pinref part="IC3" gate="G$1" pin="N/C_2"/>
+<wire x1="142.24" y1="68.58" x2="160.02" y2="68.58" width="0.1524" layer="91"/>
+<wire x1="160.02" y1="68.58" x2="160.02" y2="114.3" width="0.1524" layer="91"/>
+<wire x1="160.02" y1="114.3" x2="157.48" y2="114.3" width="0.1524" layer="91"/>
+<pinref part="C12" gate="G$1" pin="2"/>
+<junction x="142.24" y="68.58"/>
+<wire x1="76.2" y1="119.38" x2="76.2" y2="116.84" width="0.1524" layer="91"/>
+<junction x="76.2" y="116.84"/>
+<pinref part="CMP_BRKOUT" gate="G$1" pin="9"/>
+<wire x1="76.2" y1="114.3" x2="76.2" y2="109.22" width="0.1524" layer="91"/>
+<wire x1="76.2" y1="109.22" x2="78.74" y2="109.22" width="0.1524" layer="91"/>
+<wire x1="78.74" y1="109.22" x2="119.38" y2="109.22" width="0.1524" layer="91"/>
+<pinref part="C21" gate="G$1" pin="1"/>
+<wire x1="119.38" y1="93.98" x2="119.38" y2="109.22" width="0.1524" layer="91"/>
+<pinref part="IC3" gate="G$1" pin="N/C_1"/>
+<wire x1="119.38" y1="109.22" x2="119.38" y2="114.3" width="0.1524" layer="91"/>
+<wire x1="119.38" y1="114.3" x2="121.92" y2="114.3" width="0.1524" layer="91"/>
+<junction x="119.38" y="109.22"/>
+<wire x1="76.2" y1="116.84" x2="76.2" y2="114.3" width="0.1524" layer="91"/>
+<junction x="76.2" y="114.3"/>
 </segment>
 </net>
@@
 <wire x1="91.44" y1="124.46" x2="96.52" y2="124.46" width="0.1524" layer="91"/>
 <wire x1="96.52" y1="124.46" x2="96.52" y2="76.2" width="0.1524" layer="91"/>
+<wire x1="91.44" y1="124.46" x2="91.44" y2="129.54" width="0.1524" layer="91"/>
+<junction x="91.44" y="124.46"/>
+<pinref part="CMP_BRKOUT" gate="G$1" pin="1"/>
+<wire x1="76.2" y1="124.46" x2="76.2" y2="129.54" width="0.1524" layer="91"/>
+<wire x1="76.2" y1="129.54" x2="76.2" y2="157.48" width="0.1524" layer="91"/>
+<wire x1="76.2" y1="157.48" x2="139.7" y2="157.48" width="0.1524" layer="91"/>
+<pinref part="IC3" gate="G$1" pin="VDD"/>
+<wire x1="139.7" y1="157.48" x2="139.7" y2="147.32" width="0.1524" layer="91"/>
+<pinref part="C11" gate="G$1" pin="1"/>
+<wire x1="139.7" y1="157.48" x2="144.78" y2="157.48" width="0.1524" layer="91"/>
+<junction x="139.7" y="157.48"/>
+<wire x1="144.78" y1="157.48" x2="157.48" y2="157.48" width="0.1524" layer="91"/>
+<junction x="144.78" y="157.48"/>
+<pinref part="IC3" gate="G$1" pin="A1"/>
+<wire x1="157.48" y1="119.38" x2="162.56" y2="119.38" width="0.1524" layer="91"/>
+<wire x1="162.56" y1="119.38" x2="162.56" y2="121.92" width="0.1524" layer="91"/>
+<wire x1="162.56" y1="121.92" x2="162.56" y2="157.48" width="0.1524" layer="91"/>
+<wire x1="162.56" y1="157.48" x2="157.48" y2="157.48" width="0.1524" layer="91"/>
+<pinref part="IC3" gate="G$1" pin="A0"/>
+<wire x1="157.48" y1="121.92" x2="162.56" y2="121.92" width="0.1524" layer="91"/>
+<junction x="162.56" y="121.92"/>
+<wire x1="91.44" y1="129.54" x2="76.2" y2="129.54" width="0.1524" layer="91"/>
+<junction x="76.2" y="129.54"/>
 </segment>
 </net>
@@
 </segment>
 </net>
-<net name="N$31" class="0">
-<segment>
-<pinref part="CMP_BRKOUT" gate="G$1" pin="5"/>
-<wire x1="76.2" y1="119.38" x2="66.04" y2="119.38" width="0.1524" layer="91"/>
-<wire x1="66.04" y1="119.38" x2="66.04" y2="83.82" width="0.1524" layer="91"/>
-<wire x1="66.04" y1="83.82" x2="66.04" y2="66.04" width="0.1524" layer="91"/>
-<wire x1="66.04" y1="66.04" x2="162.56" y2="66.04" width="0.1524" layer="91"/>
-<pinref part="IC3" gate="G$1" pin="N/C_3"/>
-<wire x1="162.56" y1="66.04" x2="162.56" y2="116.84" width="0.1524" layer="91"/>
-<wire x1="162.56" y1="116.84" x2="157.48" y2="116.84" width="0.1524" layer="91"/>
-</segment>
-</net>
-<net name="N$32" class="0">
-<segment>
-<pinref part="CMP_BRKOUT" gate="G$1" pin="7"/>
-<wire x1="76.2" y1="116.84" x2="68.58" y2="116.84" width="0.1524" layer="91"/>
-<wire x1="68.58" y1="116.84" x2="68.58" y2="83.82" width="0.1524" layer="91"/>
-<wire x1="68.58" y1="83.82" x2="68.58" y2="68.58" width="0.1524" layer="91"/>
-<wire x1="68.58" y1="68.58" x2="142.24" y2="68.58" width="0.1524" layer="91"/>
-<pinref part="IC3" gate="G$1" pin="N/C_2"/>
-<wire x1="142.24" y1="68.58" x2="160.02" y2="68.58" width="0.1524" layer="91"/>
-<wire x1="160.02" y1="68.58" x2="160.02" y2="114.3" width="0.1524" layer="91"/>
-<wire x1="160.02" y1="114.3" x2="157.48" y2="114.3" width="0.1524" layer="91"/>
-<pinref part="C12" gate="G$1" pin="2"/>
-<junction x="142.24" y="68.58"/>
-</segment>
-</net>
-<net name="N$33" class="0">
-<segment>
-<pinref part="CMP_BRKOUT" gate="G$1" pin="9"/>
-<wire x1="76.2" y1="114.3" x2="76.2" y2="109.22" width="0.1524" layer="91"/>
-<wire x1="76.2" y1="109.22" x2="78.74" y2="109.22" width="0.1524" layer="91"/>
-<wire x1="78.74" y1="109.22" x2="119.38" y2="109.22" width="0.1524" layer="91"/>
-<pinref part="C21" gate="G$1" pin="1"/>
-<wire x1="119.38" y1="93.98" x2="119.38" y2="109.22" width="0.1524" layer="91"/>
-<pinref part="IC3" gate="G$1" pin="N/C_1"/>
-<wire x1="119.38" y1="109.22" x2="119.38" y2="114.3" width="0.1524" layer="91"/>
-<wire x1="119.38" y1="114.3" x2="121.92" y2="114.3" width="0.1524" layer="91"/>
-<junction x="119.38" y="109.22"/>
-</segment>
-</net>
