File: PCB.sch (EAGLE design)
At the start: 152 parts, among them IC3 MLX90393ELW-ABA-011-SP, IC5 STM32F407VGT6, Q11 8Mhz

Commit message: update
Connections:
- net N$21 renamed GND_BREAKOUT
- net N$30 renamed VDD_BREAKOUT
Changed lines of the file:
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@@
 </busses>
 <nets>
-<net name="N$21" class="0">
+<net name="GND_BREAKOUT" class="0">
 <segment>
 <pinref part="IC3" gate="G$1" pin="VSS"/>
@@
 <wire x1="76.2" y1="116.84" x2="76.2" y2="114.3" width="0.1524" layer="91"/>
 <junction x="76.2" y="114.3"/>
+<label x="66.04" y="99.06" size="1.778" layer="95" rot="R90"/>
 </segment>
 </net>
@@
 </segment>
 </net>
-<net name="N$30" class="0">
+<net name="VDD_BREAKOUT" class="0">
 <segment>
 <pinref part="IC3" gate="G$1" pin="VDD_IO"/>
@@
 <wire x1="91.44" y1="129.54" x2="76.2" y2="129.54" width="0.1524" layer="91"/>
 <junction x="76.2" y="129.54"/>
+<label x="76.2" y="137.16" size="1.778" layer="95" rot="R90"/>
 </segment>
 </net>

Commit message: ready for submission
Parts:
- added C15, C16, C17, C19, C20, C6, C7, C8, C9: 22nF, eagle-ltspice:C
- R17, R23, R29: value 180k -> 18k
Connections:
- net GND: now also C15.2, C16.2, C17.2, C19.2, C20.2, C6.2, C7.2, C8.2, C9.2
- net MOTOR_L_CELL1: now also C16.1
- net MOTOR_L_CELL2: now also C15.1
- net MOTOR_L_CELL3: now also C9.1
- net MOTOR_R_CELL1: now also C20.1
- net MOTOR_R_CELL2: now also C19.1
- net MOTOR_R_CELL3: now also C17.1
- net PCB_CELL1: now also C8.1
- net PCB_CELL2: now also C7.1
- net PCB_CELL3: now also C6.1
