File: PCB Overview.sch (EAGLE design)
At the start: 152 parts, among them IC3 MLX90393ELW-ABA-011-SP, IC5 STM32F407VGT6, Q11 8Mhz

Commit message: update
Parts:
- removed BOOT0, CON_SW, LASR_SW, LDR_SW, LM_SW, NRST, RASPI_SW, RM_SW: IRF512, transistor-power:IRF512
- removed C1, C2, C3, C4: 100uF, rcl:CPOL-US140CLH-0810
- removed C10: 10uF, resistor:C-EUC0805
- removed C11, C12: 10uF, resistor:C-EUC1206
- removed C13, C14: 0.1uF, resistor:C-EUC1206
- removed C18: 22uF, resistor:C-EUC0805
- removed C21, C22: 10pF, resistor:C-EUC1206
- removed C25, C30, C31, C38, C41, C42, C43, C44, C45, C5: 100nF, rcl:C-EUC0805
- removed C26: 10uF, rcl:C-EUC0805
- removed C32, C33: 2.2uF, rcl:C-EUC0805
- removed C34, C35: 1uF, rcl:C-EUC0805
- removed C39, C40: 20pF, rcl:C-EUC0805
- removed CMP_BRKOUT, COMPASS_HEADER: (no value), SparkFun-Connectors:CONN_05X2SHD
- removed CONVPOW, DCIN, DCOUT, PCBPOWER, PCB_SW, SOLAR: PRT-10474, PRT-10474:PRT-10474
- removed CONV_SW_REG, LTE_SW_REG, MICRO_SW_REG, RASPI_SW_REG: OKI-78SR-5_1.5-W36-C, OKI-78SR-5_1.5-W36-C:OKI-78SR-5_1.5-W36-C
- removed D1, D3: V60D45C-M3_I, V60D45C-M3_I:V60D45C-M3_I
- removed ESP8266_HEADER: (no value), con-lstb:MA04-2
- removed ESP_DEBUG: (no value), con-lstb:MA08-1
- removed GPS_DEBUG: (no value), con-lstb:MA06-1
- removed GPS_HEADER: (no value), con-amp:MTA04-100
- removed IC3, SPI_CMP: MLX90393ELW-ABA-011-SP, MLX90393ELW-ABA-011-SP:MLX90393ELW-ABA-011-SP
- removed IC5: STM32F407VGT6, STM32F407VGT6:STM32F407VGT6
- removed JP1, JP2, JP3, JP4, JP5: (no value), jumper:JP2E
- removed L1: FB_1206, rc-master-smd:FB_1206
- removed LASER_HEADER, LDR_HEADER: (no value), con-amp:MTA10-100
- removed LDR0, LDR1, LDR2, LDR3, LDR4, L_CELL1, L_CELL2, PCB1, PCB2, R_CELL1, R_CELL2: TPSQB2,54, testpad:TPSQB2,54
- removed LED1: BLUE, led:LEDCHIPLED_0805
- removed LEFT_MOTOR, RIGHT_MOTOR: (no value), AMP_MTA:MTA05-100
- removed LTE_PWR: LTE Modem Power Supply, MOLEX_USB:105057-0001
- removed L_CELL3, PCB3, R_CELL3: PCB_CELL3, testpad:TPSQB2,54
- removed MICRO_REG: AMS1117-3.3, AMS1117-3.3:AMS1117-3.3
- removed MOTOR_L_SENSE_IN: MOTOR_L_SENSE_IN, bt_con-jst-xh:04-JST-B4B-XH-A
- removed MOTOR_L_SENSE_OUT, MOTOR_R_SENSE_OUT: MOTOR_R_SENSE_OUT, bt_con-jst-xh:04-JST-B4B-XH-A
- removed MOTOR_R_SENSE_IN: MOTOR_R_SENSE_IN, bt_con-jst-xh:04-JST-B4B-XH-A
- removed PCB_SENSE_IN: PCB_SENSE_IN, bt_con-jst-xh:04-JST-B4B-XH-A
- removed PCB_SENSE_OUT: PCB_SENSE_OUT, bt_con-jst-xh:04-JST-B4B-XH-A
- removed PWR, RST: RED, led:LEDCHIPLED_0805
- removed Q11: 8Mhz, special:XTAL/S
- removed R1: 43k, resistor:R-US_R0805
- removed R10, R9: 10K, resistor:R-US_R1206
- removed R11: 47, rcl:R-US_R0805
- removed R12, R50, R52: 100K, rcl:R-US_R0805
- removed R13, R35, R51: 510, rcl:R-US_R0805
- removed R14, R36, R47, R49: 10K, rcl:R-US_R0805
- removed R15: 100k, resistor:R-US_R0805
- removed R16: 10k, resistor:R-US_R0805
- removed R17, R23, R29: 180k, resistor:R-US_R0805
- removed R18, R24, R30: 6.2k, resistor:R-US_R0805
- removed R19, R25, R31: 8.2k, resistor:R-US_R0805
- removed R2, R8: 51k, resistor:R-US_R0805
- removed R20, R26, R32: 5.1k, resistor:R-US_R0805
- removed R21, R27, R33: 680, resistor:R-US_R0805
- removed R22, R28, R34: 2.4k, resistor:R-US_R0805
- removed R3: 43K, resistor:R-US_R0805
- removed R37, R39, R40, R41, R42, R46, R53, R54, R55: 100k, resistor:R-US_R1206
- removed R38: 220, rcl:R-US_R0805
- removed R4, R6: 51K, resistor:R-US_R0805
- removed R43, R44: 1M, resistor:R-US_R0805
- removed R45, R48, R56: 200, rcl:R-US_R0805
- removed R5: 75K, resistor:R-US_R0805
- removed R7: 75k, resistor:R-US_R0805
- removed RASPI_PWR: Raspi Power Supply, MOLEX_USB:105057-0001
- removed STLINK: (no value), pinhead:PINHD-1X6
- added BOOT1, CON_SW1, LASR_SW1, LDR_SW1, LM_SW1, NRST1, RASPI_SW1, RM_SW1: IRF512, transistor-power:IRF512
- added C15, C16, C8, C9: 100uF, rcl:CPOL-US140CLH-0810
- added C17, C20, C23, C36, C47, C48, C49, C50, C51, C52: 100nF, rcl:C-EUC0805
- added C19: 10uF, rcl:C-EUC0805
- added C24, C27: 2.2uF, rcl:C-EUC0805
- added C28, C29: 1uF, rcl:C-EUC0805
- added C37, C46: 20pF, rcl:C-EUC0805
- added C53, C54: 10uF, resistor:C-EUC1206
- added C55, C56: 10pF, resistor:C-EUC1206
- added C57, C58: 0.1uF, resistor:C-EUC1206
- added C6: 10uF, resistor:C-EUC0805
- added C7: 22uF, resistor:C-EUC0805
- added CMP_BRKOUT1, COMPASS_HEADER1: (no value), SparkFun-Connectors:CONN_05X2SHD
- added CONVPOW1, DCIN1, DCOUT1, PCBPOWER1, PCB_SW1, SOLAR1: PRT-10474, PRT-10474:PRT-10474
- added CONV_SW_REG1, LTE_SW_REG1, MICRO_SW_REG1, RASPI_SW_REG1: OKI-78SR-5_1.5-W36-C, OKI-78SR-5_1.5-W36-C:OKI-78SR-5_1.5-W36-C
- added D2, D4: V60D45C-M3_I, V60D45C-M3_I:V60D45C-M3_I
- added ESP8266_HEADER1: (no value), con-lstb:MA04-2
- added ESP_DEBUG1: (no value), con-lstb:MA08-1
- added GPS_DEBUG1: (no value), con-lstb:MA06-1
- added GPS_HEADER1: (no value), con-amp:MTA04-100
- added IC1: STM32F407VGT6, STM32F407VGT6:STM32F407VGT6
- added IC2, SPI_CMP1: MLX90393ELW-ABA-011-SP, MLX90393ELW-ABA-011-SP:MLX90393ELW-ABA-011-SP
- added JP10, JP6, JP7, JP8, JP9: (no value), jumper:JP2E
- added L2: FB_1206, rc-master-smd:FB_1206
- added LASER_HEADER1, LDR_HEADER1: (no value), con-amp:MTA10-100
- added LDR5, LDR6, LDR7, LDR8, LDR9, L_CELL5, L_CELL6, PCB5, PCB6, R_CELL5, R_CELL6: TPSQB2,54, testpad:TPSQB2,54
- added LED2: BLUE, led:LEDCHIPLED_0805
- added LEFT_MOTOR1, RIGHT_MOTOR1: (no value), AMP_MTA:MTA05-100
- added LTE_PWR1: LTE Modem Power Supply, MOLEX_USB:105057-0001
- added L_CELL4, PCB4, R_CELL4: PCB_CELL3, testpad:TPSQB2,54
- added MICRO_REG1: AMS1117-3.3, AMS1117-3.3:AMS1117-3.3
- added MOTOR_L_SENSE_IN1: MOTOR_L_SENSE_IN, bt_con-jst-xh:04-JST-B4B-XH-A
- added MOTOR_L_SENSE_OUT1, MOTOR_R_SENSE_OUT1: MOTOR_R_SENSE_OUT, bt_con-jst-xh:04-JST-B4B-XH-A
- added MOTOR_R_SENSE_IN1: MOTOR_R_SENSE_IN, bt_con-jst-xh:04-JST-B4B-XH-A
- added PCB_SENSE_IN1: PCB_SENSE_IN, bt_con-jst-xh:04-JST-B4B-XH-A
- added PCB_SENSE_OUT1: PCB_SENSE_OUT, bt_con-jst-xh:04-JST-B4B-XH-A
- added PWR1, RST1: RED, led:LEDCHIPLED_0805
- added Q1: 8Mhz, special:XTAL/S
- added R100, R101, R87: 200, rcl:R-US_R0805
- added R102, R105, R106, R107, R108, R109, R110, R111, R114: 100k, resistor:R-US_R1206
- added R103, R104: 10K, resistor:R-US_R1206
- added R57, R60: 51K, resistor:R-US_R0805
- added R58: 75K, resistor:R-US_R0805
- added R59: 43K, resistor:R-US_R0805
- added R61, R64: 51k, resistor:R-US_R0805
- added R62: 43k, resistor:R-US_R0805
- added R63: 75k, resistor:R-US_R0805
- added R65: 100k, resistor:R-US_R0805
- added R66: 10k, resistor:R-US_R0805
- added R67, R68: 1M, resistor:R-US_R0805
- added R69, R75, R81: 180k, resistor:R-US_R0805
- added R70, R76, R82: 6.2k, resistor:R-US_R0805
- added R71, R77, R83: 8.2k, resistor:R-US_R0805
- added R72, R78, R84: 5.1k, resistor:R-US_R0805
- added R73, R79, R85: 680, resistor:R-US_R0805
- added R74, R80, R86: 2.4k, resistor:R-US_R0805
- added R88: 47, rcl:R-US_R0805
- added R89, R97, R99: 100K, rcl:R-US_R0805
- added R90, R93, R98: 510, rcl:R-US_R0805
- added R91, R94, R95, R96: 10K, rcl:R-US_R0805
- added R92: 220, rcl:R-US_R0805
- added RASPI_PWR1: Raspi Power Supply, MOLEX_USB:105057-0001
- added STLINK1: (no value), pinhead:PINHD-1X6
Connections:
- removed net N$1: PCB_SENSE_IN-3.1, PCB_SENSE_OUT-3.1, R21.1
- removed net N$10: MOTOR_L_SENSE_IN-3.1, MOTOR_L_SENSE_OUT-3.1, R27.1
- removed net N$11: CONV_SW_REG.COMMON(GROUND), CON_SW.D, R43.2
- removed net N$12: MOTOR_L_SENSE_IN-2.1, MOTOR_L_SENSE_OUT-2.1, R25.1
- removed net N$13: R5.2, R6.1, RASPI_PWR.2
- removed net N$14: MOTOR_L_SENSE_IN-1.1, MOTOR_L_SENSE_OUT-1.1, R23.1
- removed net N$15: R3.2, R4.1, RASPI_PWR.3
- removed net N$16: C2.+, R3.1, R5.1, RASPI_PWR.1, RASPI_SW_REG.POSITIVE_OUTPUT
- removed net N$17: MOTOR_R_SENSE_IN-3.1, MOTOR_R_SENSE_OUT-3.1, R33.1
- removed net N$19: R44.2, RASPI_SW.D, RASPI_SW_REG.COMMON(GROUND)
- removed net N$2: CONVPOW.POS, CONV_SW_REG.POSITIVE_OUTPUT
- removed net N$20: MOTOR_R_SENSE_IN-2.1, MOTOR_R_SENSE_OUT-2.1, R31.1
- removed net N$21: C11.2, C12.2, C21.1, C22.1, CMP_BRKOUT.3, CMP_BRKOUT.5, CMP_BRKOUT.7, CMP_BRKOUT.9, IC3.N/C_1, IC3.N/C_2, IC3.N/C_3, IC3.N/C_4, IC3.N/C_5, IC3.VSS
- removed net N$22: CMP_BRKOUT.4, IC3.INT
- removed net N$23: C32.2, IC5.VCAP_2
- removed net N$24: C22.2, CMP_BRKOUT.6, IC3.SCL/SCLK, R10.2
- removed net N$25: C21.2, CMP_BRKOUT.8, IC3.SDA/MOSI, R9.2
- removed net N$26: LEFT_MOTOR.4, LM_SW.D
- removed net N$27: PCB_SENSE_IN-2.1, PCB_SENSE_OUT-2.1, R19.1
- removed net N$28: MOTOR_R_SENSE_IN-1.1, MOTOR_R_SENSE_OUT-1.1, R29.1
- removed net N$29: CMP_BRKOUT.10, IC3.INT/TRIG
- removed net N$3: IC5.PB2, JP3.2
- removed net N$30: C11.1, C12.1, CMP_BRKOUT.1, CMP_BRKOUT.2, IC3.A0, IC3.A1, IC3.SENB/CS, IC3.VDD, IC3.VDD_IO, R10.1, R9.1
- removed net N$34: R56.1, RST.A
- removed net N$35: D1.CATHODE_(HEATSINK), D3.CATHODE_(HEATSINK), DCOUT.POS
- removed net N$36: C33.2, IC5.VCAP_1
- removed net N$37: PWR.A, R48.2
- removed net N$38: JP3.1, R14.2
- removed net N$39: C30.1, C35.1, IC5.VREF+, R11.1
- removed net N$4: D1.ANODE_1, D1.ANODE_2, DCIN.POS
- removed net N$40: C31.1, C34.1, IC5.VDDA, L1.1, R11.2
- removed net N$41: ESP_DEBUG.3, JP4.3
- removed net N$43: IC5.PD15, R45.1
- removed net N$44: JP2.2, NRST.G, R52.2
- removed net N$45: BOOT0.S, R51.1
- removed net N$46: GPS_DEBUG.3, JP5.1
- removed net N$47: LDR_SW.D, R37.2, R39.2, R40.2, R41.2, R42.2
- removed net N$48: ESP8266_HEADER.4, ESP8266_HEADER.8, JP4.2
- removed net N$49: GPS_HEADER.1, JP5.3
- removed net N$5: D3.ANODE_1, D3.ANODE_2, SOLAR.POS
- removed net N$50: LED1.A, R45.2
- removed net N$51: LASER_HEADER.1, LASER_HEADER.3, LASER_HEADER.5, LASER_HEADER.7, LASER_HEADER.9, LASR_SW.D
- removed net N$52: PCBPOWER.POS, PCB_SW.GND
- removed net N$6: C1.+, LTE_PWR.1, LTE_SW_REG.POSITIVE_OUTPUT, R1.1, R7.1
- removed net N$63: C5.1, IC5.NRST, R12.2, R56.2
- removed net N$65: IC5.PH1, R38.1
- removed net N$66: IC5.BOOT0, JP1.2
- removed net N$67: JP1.1, R35.2
- removed net N$68: C39.1, Q11.2, R38.2
- removed net N$69: BOOT0.D, JP1.3, R36.1
- removed net N$7: LTE_PWR.3, R1.2, R2.1
- removed net N$70: C40.1, IC5.PH0, Q11.1
- removed net N$73: RIGHT_MOTOR.4, RM_SW.D
- removed net N$8: PCB_SENSE_IN-1.1, PCB_SENSE_OUT-1.1, R17.1
- removed net N$83: JP3.3, R13.2
- removed net N$9: LTE_PWR.2, R7.2, R8.1
- new net N$100: R101.1, RST1.A
- new net N$101: LASER_HEADER1.1, LASER_HEADER1.3, LASER_HEADER1.5, LASER_HEADER1.7, LASER_HEADER1.9, LASR_SW1.D
- new net N$102: C53.2, C54.2, C55.1, C56.1, CMP_BRKOUT1.3, CMP_BRKOUT1.5, CMP_BRKOUT1.7, CMP_BRKOUT1.9, IC2.N/C_1, IC2.N/C_2, IC2.N/C_3, IC2.N/C_4, IC2.N/C_5, IC2.VSS
- new net N$103: CMP_BRKOUT1.4, IC2.INT
- new net N$104: CMP_BRKOUT1.10, IC2.INT/TRIG
- new net N$105: C53.1, C54.1, CMP_BRKOUT1.1, CMP_BRKOUT1.2, IC2.A0, IC2.A1, IC2.SENB/CS, IC2.VDD, IC2.VDD_IO, R103.1, R104.1
- new net N$106: C56.2, CMP_BRKOUT1.6, IC2.SCL/SCLK, R104.2
- new net N$107: C55.2, CMP_BRKOUT1.8, IC2.SDA/MOSI, R103.2
- new net N$108: GPS_DEBUG1.3, JP9.1
- new net N$109: GPS_HEADER1.1, JP9.3
- new net N$110: LEFT_MOTOR1.4, LM_SW1.D
- new net N$113: RIGHT_MOTOR1.4, RM_SW1.D
- new net N$118: LDR_SW1.D, R107.2, R108.2, R109.2, R110.2, R111.2
- new net N$119: ESP8266_HEADER1.4, ESP8266_HEADER1.8, JP10.2
- new net N$123: ESP_DEBUG1.3, JP10.3
- new net N$18: LTE_PWR1.3, R61.1, R62.2
- new net N$31: LTE_PWR1.2, R63.2, R64.1
- new net N$32: R59.2, R60.1, RASPI_PWR1.3
- new net N$33: CONVPOW1.POS, CONV_SW_REG1.POSITIVE_OUTPUT
- new net N$42: C9.+, R58.1, R59.1, RASPI_PWR1.1, RASPI_SW_REG1.POSITIVE_OUTPUT
- new net N$53: R57.1, R58.2, RASPI_PWR1.2
- new net N$54: C8.+, LTE_PWR1.1, LTE_SW_REG1.POSITIVE_OUTPUT, R62.1, R63.1
- new net N$55: R68.2, RASPI_SW1.D, RASPI_SW_REG1.COMMON(GROUND)
- new net N$56: PCBPOWER1.POS, PCB_SW1.GND
- new net N$57: CONV_SW_REG1.COMMON(GROUND), CON_SW1.D, R67.2
- new net N$58: D2.ANODE_1, D2.ANODE_2, DCIN1.POS
- new net N$59: D4.ANODE_1, D4.ANODE_2, SOLAR1.POS
- new net N$60: D2.CATHODE_(HEATSINK), D4.CATHODE_(HEATSINK), DCOUT1.POS
- new net N$61: PCB_SENSE_IN1-3.1, PCB_SENSE_OUT1-3.1, R73.1
- new net N$62: PCB_SENSE_IN1-1.1, PCB_SENSE_OUT1-1.1, R69.1
- new net N$64: PCB_SENSE_IN1-2.1, PCB_SENSE_OUT1-2.1, R71.1
- new net N$74: MOTOR_L_SENSE_IN1-3.1, MOTOR_L_SENSE_OUT1-3.1, R79.1
- new net N$75: MOTOR_L_SENSE_IN1-2.1, MOTOR_L_SENSE_OUT1-2.1, R77.1
- new net N$76: MOTOR_L_SENSE_IN1-1.1, MOTOR_L_SENSE_OUT1-1.1, R75.1
- new net N$77: MOTOR_R_SENSE_IN1-3.1, MOTOR_R_SENSE_OUT1-3.1, R85.1
- new net N$78: MOTOR_R_SENSE_IN1-2.1, MOTOR_R_SENSE_OUT1-2.1, R83.1
- new net N$79: MOTOR_R_SENSE_IN1-1.1, MOTOR_R_SENSE_OUT1-1.1, R81.1
- new net N$80: PWR1.A, R87.2
- new net N$81: C27.2, IC1.VCAP_1
- new net N$82: C24.2, IC1.VCAP_2
- new net N$84: C52.1, IC1.NRST, R101.2, R89.2
- new net N$85: JP6.2, NRST1.G, R99.2
- new net N$86: IC1.BOOT0, JP7.2
- new net N$87: BOOT1.D, JP7.3, R91.1
- new net N$88: JP7.1, R90.2
- new net N$89: IC1.PH1, R92.1
- new net N$90: C37.1, Q1.2, R92.2
- new net N$91: C46.1, IC1.PH0, Q1.1
- new net N$92: IC1.PB2, JP8.2
- new net N$93: JP8.1, R94.2
- new net N$94: JP8.3, R93.2
- new net N$95: BOOT1.S, R98.1
- new net N$96: IC1.PD15, R100.1
- new net N$97: LED2.A, R100.2
- new net N$98: C20.1, C29.1, IC1.VREF+, R88.1
- new net N$99: C23.1, C28.1, IC1.VDDA, L2.1, R88.2
- net CMP_INT: now also COMPASS_HEADER1.4, IC1.PE9; no longer COMPASS_HEADER.4, IC5.PE9
- net CMP_MISO: now also IC1.PB14, SPI_CMP1.MISO; no longer IC5.PB14, SPI_CMP.MISO
- net CMP_MOSI: now also IC1.PB15, SPI_CMP1.SDA/MOSI; no longer IC5.PB15, SPI_CMP.SDA/MOSI
- net CMP_SCL: now also COMPASS_HEADER1.6, IC1.PB8, R95.1; no longer COMPASS_HEADER.6, IC5.PB8, R47.1
- net CMP_SCLK: now also IC1.PB13, SPI_CMP1.SCL/SCLK; no longer IC5.PB13, SPI_CMP.SCL/SCLK
- net CMP_SDA: now also COMPASS_HEADER1.8, IC1.PB9, R96.1; no longer COMPASS_HEADER.8, IC5.PB9, R49.1
- net CMP_SPI_INT: now also IC1.PE7, SPI_CMP1.INT; no longer IC5.PE7, SPI_CMP.INT
- net CMP_TRG: now also COMPASS_HEADER1.10, IC1.PE10; no longer COMPASS_HEADER.10, IC5.PE10
- net CMP_TRIG: now also IC1.PE8, SPI_CMP1.INT/TRIG; no longer IC5.PE8, SPI_CMP.INT/TRIG
- net C_MOS: now also CON_SW1.G, IC1.PA10, R65.2; no longer CON_SW.G, IC5.PA10, R15.2
- net ESP_GPIO0: now also ESP8266_HEADER1.5, ESP_DEBUG1.8, JP6.3; no longer ESP8266_HEADER.5, ESP_DEBUG.8, JP2.3
- net ESP_GPIO2: now also BOOT1.G, ESP8266_HEADER1.3, ESP_DEBUG1.7, R97.2; no longer BOOT0.G, ESP8266_HEADER.3, ESP_DEBUG.7, R50.2
- net ESP_RX: now also ESP8266_HEADER1.7, ESP_DEBUG1.4, IC1.PB10; no longer ESP8266_HEADER.7, ESP_DEBUG.4, IC5.PB10
- net ESP_TX: now also ESP8266_HEADER1.2, ESP_DEBUG1.5, IC1.PB11; no longer ESP8266_HEADER.2, ESP_DEBUG.5, IC5.PB11
- net GND: now also C15.-, C16.-, C17.2, C19.2, C20.2, C23.2, C24.1, C27.1, C28.2, C29.2, C36.1, C37.2, C46.2, C47.2, C48.2, C49.2, C50.2, C51.2, C52.2, C57.1, C58.2, C6.2, C7.2, C8.-, C9.-, COMPASS_HEADER1.3, COMPASS_HEADER1.5, COMPASS_HEADER1.7, COMPASS_HEADER1.9, CONVPOW1.GND, CON_SW1.S, DCIN1.GND, DCOUT1.GND, ESP8266_HEADER1.1, ESP_DEBUG1.1, GPS_DEBUG1.1, GPS_HEADER1.4, IC1.VSS, IC1.VSSA, LASR_SW1.S, LDR_SW1.S, LED2.C, LEFT_MOTOR1.3, LEFT_MOTOR1.5, LM_SW1.S, LTE_PWR1.4, LTE_SW_REG1.COMMON(GROUND), MICRO_REG1.ADJ/GND, MICRO_SW_REG1.COMMON(GROUND), MOTOR_L_SENSE_IN1-4.1, MOTOR_L_SENSE_OUT1-4.1, MOTOR_R_SENSE_IN1-4.1, MOTOR_R_SENSE_OUT1-4.1, NRST1.S, PCBPOWER1.GND, PCB_SENSE_IN1-4.1, PCB_SENSE_OUT1-4.1, PWR1.C, R105.1, R106.1, R57.2, R60.2, R61.2, R64.2, R65.1, R70.2, R72.2, R74.2, R76.2, R78.2, R80.2, R82.2, R84.2, R86.2, R90.1, R93.1, R97.1, R98.2, RASPI_PWR1.4, RASPI_SW1.S, RIGHT_MOTOR1.3, RIGHT_MOTOR1.5, RM_SW1.S, SOLAR1.GND, SPI_CMP1.A0, SPI_CMP1.A1, SPI_CMP1.N/C_1, SPI_CMP1.N/C_2, SPI_CMP1.N/C_3, SPI_CMP1.N/C_4, SPI_CMP1.N/C_5, SPI_CMP1.SENB/CS, SPI_CMP1.VSS, STLINK1.3; no longer C1.-, C10.2, C13.1, C14.2, C18.2, C2.-, C25.2, C26.2, C3.-, C30.2, C31.2, C32.1, C33.1, C34.2, C35.2, C38.1, C39.2, C4.-, C40.2, C41.2, C42.2, C43.2, C44.2, C45.2, C5.2, COMPASS_HEADER.3, COMPASS_HEADER.5, COMPASS_HEADER.7, COMPASS_HEADER.9, CONVPOW.GND, CON_SW.S, DCIN.GND, DCOUT.GND, ESP8266_HEADER.1, ESP_DEBUG.1, GPS_DEBUG.1, GPS_HEADER.4, IC5.VSS, IC5.VSSA, LASR_SW.S, LDR_SW.S, LED1.C, LEFT_MOTOR.3, LEFT_MOTOR.5, LM_SW.S, LTE_PWR.4, LTE_SW_REG.COMMON(GROUND), MICRO_REG.ADJ/GND, MICRO_SW_REG.COMMON(GROUND), MOTOR_L_SENSE_IN-4.1, MOTOR_L_SENSE_OUT-4.1, MOTOR_R_SENSE_IN-4.1, MOTOR_R_SENSE_OUT-4.1, NRST.S, PCBPOWER.GND, PCB_SENSE_IN-4.1, PCB_SENSE_OUT-4.1, PWR.C, R13.1, R15.1, R18.2, R2.2, R20.2, R22.2, R24.2, R26.2, R28.2, R30.2, R32.2, R34.2, R35.1, R4.2, R46.1, R50.1, R51.2, R53.1, R6.2, R8.2, RASPI_PWR.4, RASPI_SW.S, RIGHT_MOTOR.3, RIGHT_MOTOR.5, RM_SW.S, SOLAR.GND, SPI_CMP.A0, SPI_CMP.A1, SPI_CMP.N/C_1, SPI_CMP.N/C_2, SPI_CMP.N/C_3, SPI_CMP.N/C_4, SPI_CMP.N/C_5, SPI_CMP.SENB/CS, SPI_CMP.VSS, STLINK.3
- net GPS_RX: now also GPS_DEBUG1.4, GPS_HEADER1.2, IC1.PB6; no longer GPS_DEBUG.4, GPS_HEADER.2, IC5.PB6
- net GPS_TX: now also GPS_DEBUG1.5, GPS_HEADER1.3, IC1.PB7; no longer GPS_DEBUG.5, GPS_HEADER.3, IC5.PB7
- net LASER_MOS: now also IC1.PA12, LASR_SW1.G, R102.1; no longer IC5.PA12, LASR_SW.G, R55.1
- net LDR0: now also IC1.PA0, LDR9.TP, LDR_HEADER1.2, R107.1; no longer IC5.PA0, LDR0.TP, LDR_HEADER.2, R37.1
- net LDR1: now also IC1.PA1, LDR8.TP, LDR_HEADER1.4, R108.1; no longer IC5.PA1, LDR1.TP, LDR_HEADER.4, R39.1
- net LDR2: now also IC1.PA2, LDR7.TP, LDR_HEADER1.6, R109.1; no longer IC5.PA2, LDR2.TP, LDR_HEADER.6, R40.1
- net LDR3: now also IC1.PA3, LDR6.TP, LDR_HEADER1.8, R110.1; no longer IC5.PA3, LDR3.TP, LDR_HEADER.8, R41.1
- net LDR4: now also IC1.PA4, LDR5.TP, LDR_HEADER1.10, R111.1; no longer IC5.PA4, LDR4.TP, LDR_HEADER.10, R42.1
- net LDR_MOS: now also IC1.PA15, LDR_SW1.G, R114.1; no longer IC5.PA15, LDR_SW.G, R54.1
- net L_MOS: now also IC1.PA8, LM_SW1.G, R105.2; no longer IC5.PA8, LM_SW.G, R46.2
- net L_PWM: now also IC1.PC6, LEFT_MOTOR1.1; no longer IC5.PC6, LEFT_MOTOR.1
- net MOTOR_L_CELL1: now also IC1.PB0, L_CELL6.TP, R79.2, R80.1; no longer IC5.PB0, L_CELL1.TP, R27.2, R28.1
- net MOTOR_L_CELL2: now also IC1.PB1, L_CELL5.TP, R77.2, R78.1; no longer IC5.PB1, L_CELL2.TP, R25.2, R26.1
- net MOTOR_L_CELL3: now also IC1.PC0, L_CELL4.TP, R75.2, R76.1; no longer IC5.PC0, L_CELL3.TP, R23.2, R24.1
- net MOTOR_R_CELL1: now also IC1.PC1, R85.2, R86.1, R_CELL6.TP; no longer IC5.PC1, R33.2, R34.1, R_CELL1.TP
- net MOTOR_R_CELL2: now also IC1.PC2, R83.2, R84.1, R_CELL5.TP; no longer IC5.PC2, R31.2, R32.1, R_CELL2.TP
- net MOTOR_R_CELL3: now also IC1.PC3, R81.2, R82.1, R_CELL4.TP; no longer IC5.PC3, R29.2, R30.1, R_CELL3.TP
- net NRST: now also NRST1.D, RST1.C, STLINK1.5; no longer NRST.D, RST.C, STLINK.5
- net PCB_CELL1: now also IC1.PA5, PCB6.TP, R73.2, R74.1; no longer IC5.PA5, PCB1.TP, R21.2, R22.1
- net PCB_CELL2: now also IC1.PA6, PCB5.TP, R71.2, R72.1; no longer IC5.PA6, PCB2.TP, R19.2, R20.1
- net PCB_CELL3: now also IC1.PA7, PCB4.TP, R69.2, R70.1; no longer IC5.PA7, PCB3.TP, R17.2, R18.1
- net RASPI_MOS: now also IC1.PA11, R66.2, RASPI_SW1.G; no longer IC5.PA11, R16.2, RASPI_SW.G
- net R_MOS: now also IC1.PA9, R106.2, RM_SW1.G; no longer IC5.PA9, R53.2, RM_SW.G
- net R_PWM: now also IC1.PC7, RIGHT_MOTOR1.1; no longer IC5.PC7, RIGHT_MOTOR.1
- net SWCLK: now also IC1.PA14, STLINK1.2; no longer IC5.PA14, STLINK.2
- net SWDIO: now also IC1.PA13, STLINK1.4; no longer IC5.PA13, STLINK.4
- net SWO: now also IC1.PB3, STLINK1.6; no longer IC5.PB3, STLINK.6
- net VBAT: now also CONV_SW_REG1.POSITIVE_INPUT, LTE_SW_REG1.POSITIVE_INPUT, MICRO_SW_REG1.POSITIVE_INPUT, PCB_SW1.POS, R66.1, R67.1, R68.1, RASPI_SW_REG1.POSITIVE_INPUT; no longer CONV_SW_REG.POSITIVE_INPUT, LTE_SW_REG.POSITIVE_INPUT, MICRO_SW_REG.POSITIVE_INPUT, PCB_SW.POS, R16.1, R43.1, R44.1, RASPI_SW_REG.POSITIVE_INPUT
- net VCC: now also C16.+, C17.1, C19.1, C36.2, C47.1, C48.1, C49.1, C50.1, C51.1, C57.2, C58.1, C7.1, COMPASS_HEADER1.1, COMPASS_HEADER1.2, IC1.VBAT, IC1.VDD, JP10.1, JP6.1, JP9.2, L2.2, MICRO_REG1.VOUT, R102.2, R114.2, R87.1, R89.1, R91.2, R94.1, R95.2, R96.2, R99.1, SPI_CMP1.VDD, SPI_CMP1.VDD_IO, STLINK1.1; no longer C13.2, C14.1, C18.1, C25.1, C26.1, C38.2, C4.+, C41.1, C42.1, C43.1, C44.1, C45.1, COMPASS_HEADER.1, COMPASS_HEADER.2, IC5.VBAT, IC5.VDD, JP2.1, JP4.1, JP5.2, L1.2, MICRO_REG.VOUT, R12.1, R14.1, R36.2, R47.2, R48.1, R49.2, R52.1, R54.2, R55.2, SPI_CMP.VDD, SPI_CMP.VDD_IO, STLINK.1
- net VDD: now also C15.+, C6.1, LASER_HEADER1.10, LASER_HEADER1.2, LASER_HEADER1.4, LASER_HEADER1.6, LASER_HEADER1.8, LDR_HEADER1.1, LDR_HEADER1.3, LDR_HEADER1.5, LDR_HEADER1.7, LDR_HEADER1.9, MICRO_REG1.VIN, MICRO_SW_REG1.POSITIVE_OUTPUT; no longer C10.1, C3.+, LASER_HEADER.10, LASER_HEADER.2, LASER_HEADER.4, LASER_HEADER.6, LASER_HEADER.8, LDR_HEADER.1, LDR_HEADER.3, LDR_HEADER.5, LDR_HEADER.7, LDR_HEADER.9, MICRO_REG.VIN, MICRO_SW_REG.POSITIVE_OUTPUT
Other:
- note added: "Compass Breakout Board"
- note added: "GPS Header and Debugger"
- note added: "Left Motor Controller"
- note added: "Onboard Compass Module"
- note added: "Right Motor Controller"
