File: PCB.brd (EAGLE design)
At the start: 78.7 x 272.7 mm, 153 parts, among them IC3 MLX90393ELW-ABA-011-SP, IC5 STM32F407VGT6, Q10 2N3906, Q11 8Mhz, Q12 2N3906, Q13 2N3906, Q14 2N3906, Q15 2N3906

Commit message: update
Parts:
- GPS_HEADER: device AMP_MTA:1X09MTA -> con-amp:10X04MTA
- moved GPS_HEADER 64.8 mm to (5.08, 78.7), turned to 270 degrees
Connections:
- removed net CMP_CS: SPI_CMP.2
- removed net ESP_EN: ESP8266_HEADER.4
- removed net N$10: R16.2, RASPI_SW.G
- removed net N$13: R29.1, R30.2
- removed net N$17: R31.1, R32.2
- removed net N$19: Q15.1, R47.2
- removed net N$20: R33.1, R34.2
- removed net N$28: CON_SW.G, R15.2
- removed net N$37: R17.1, R18.2
- removed net N$42: R19.1, R20.2
- removed net N$49: R21.1, R22.2
- removed net N$52: R23.1, R24.2
- removed net N$59: R25.1, R26.2
- removed net N$62: R27.1, R28.2
- removed net N$75: Q10.1, R39.2
- removed net N$78: Q12.1, R41.2
- removed net N$80: Q13.1, R43.2
- removed net N$82: Q14.1, R45.2
- new net C_MOS: CON_SW.G, IC5.69, R15.2
- new net GPS_RX: GPS_HEADER.2, IC5.92
- new net GPS_TX: GPS_HEADER.3, IC5.93
- new net LASER_MOS: IC5.71, LASR_SW.G
- new net LDR0: IC5.23, Q10.1, R39.2
- new net LDR1: IC5.24, Q12.1, R41.2
- new net LDR2: IC5.25, Q13.1, R43.2
- new net LDR3: IC5.26, Q15.1, R47.2
- new net LDR4: IC5.29, Q14.1, R45.2
- new net LDR_MOS: IC5.77, LDR_SW.G
- new net L_MOS: IC5.67, LM_SW.G
- new net MOTOR_L_CELL1: IC5.35, R31.1, R32.2
- new net MOTOR_L_CELL2: IC5.36, R23.1, R24.2
- new net MOTOR_L_CELL3: IC5.15, R21.1, R22.2
- new net MOTOR_R_CELL1: IC5.16, R33.1, R34.2
- new net MOTOR_R_CELL2: IC5.17, R27.1, R28.2
- new net MOTOR_R_CELL3: IC5.18, R25.1, R26.2
- new net PCB_CELL1: IC5.30, R29.1, R30.2
- new net PCB_CELL2: IC5.31, R19.1, R20.2
- new net PCB_CELL3: IC5.32, R17.1, R18.2
- new net RASPI_MOS: IC5.70, R16.2, RASPI_SW.G
- new net R_MOS: IC5.68, RM_SW.G
- net CMP_INT: now also IC5.40
- net CMP_MISO: now also IC5.53
- net CMP_MOSI: now also IC5.54
- net CMP_SCL: now also IC5.95
- net CMP_SCLK: now also IC5.52
- net CMP_SDA: now also IC5.96
- net CMP_SPI_INT: now also IC5.38
- net CMP_TRG: now also IC5.41
- net CMP_TRIG: now also IC5.39
- net ESP_RX: now also IC5.47; no longer IC5.68
- net ESP_TX: now also IC5.48; no longer IC5.69
- net GND: now also GPS_HEADER.4, SPI_CMP.2
- net L_PWM: now also IC5.63
- net R_PWM: now also IC5.64
- net VCC: now also ESP8266_HEADER.4, GPS_HEADER.1

Commit message: update
Parts:
- removed C15, C16, C17, C19, C20, C5: 0.1uF, rcl:C1206
- removed MOTOR_L_CELL2, MOTOR_L_CELL3, MOTOR_R_CELL2, MOTOR_R_CELL3, PCB_CELL2, PCB_CELL3: INA148UA, INA148UA:SOIC127P600X175-8N
- removed R17, R18, R19, R20, R21, R22, R23, R24, R25, R26, R27, R28, R29, R30, R31, R32, R33, R34: 5k, resistor:R1206
- added C23: 100uF, rcl:C1206
- LTE_PWR: value LTE Model Power Supply -> LTE Modem Power Supply; device con-berg:PN87520 -> MOLEX_USB:105057-0001
- PWR: value PWR -> RED
- R15, R16: value 2.2k -> 10k
- RASPI_PWR: device con-berg:PN87520 -> MOLEX_USB:105057-0001
- RST: value RST -> RED
- moved RASPI_SW 57.2 mm to (53.5, 8.89), turned to 270 degrees
- moved R16 55.0 mm to (54.7, 10.5), flipped to the bottom, turned to 90 degrees
- moved R6 26.9 mm to (62.2, 43.2), turned to 270 degrees
- moved R4 25.4 mm to (58.4, 43.2), turned to 270 degrees
- moved RASPI_PWR 18.9 mm to (69.8, 47.0), turned to 270 degrees
- moved R5 14.5 mm to (62.2, 50.8), turned to 270 degrees
- moved LTE_PWR 12.8 mm to (50.8, 47.0)
- moved R3 11.5 mm to (58.4, 50.8), turned to 270 degrees
- moved CONVPOW 8.89 mm to (69.8, 14.0), turned to 270 degrees
- moved CON_SW 7.75 mm to (46.9, 9.02)
- moved R2 5.24 mm to (62.2, 50.8), flipped to the bottom
- moved R8 5.24 mm to (58.4, 50.8), flipped to the bottom
- moved R1 5.08 mm to (62.2, 43.2), flipped to the bottom
- moved R7 5.08 mm to (58.4, 43.2), flipped to the bottom
- moved C1 5.02 mm to (57.5, 11.9)
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Connections:
- removed net N$35: R4.2, R6.2, RASPI_PWR.4, RASPI_SW.S
- removed net N$39: PCB_CELL2.6, R19.2
- removed net N$4: PCB_CELL3.6, R17.2
- removed net N$48: MOTOR_L_CELL3.6, R21.2
- removed net N$51: MOTOR_L_CELL2.6, R23.2
- removed net N$58: MOTOR_R_CELL3.6, R25.2
- removed net N$61: MOTOR_R_CELL2.6, R27.2
- new net ADJ/GND: MICRO_REG.1
- new net N$19: RASPI_SW.S, RASPI_SW_REG.2
- net GND: now also C23.2, CONVPOW.1, R4.2, R6.2, RASPI_PWR.4; no longer CONV_SW_REG.2, MICRO_REG.1, RASPI_SW_REG.2
- net MOTOR_L_CELL1: no longer R31.1, R32.2
- net MOTOR_L_CELL2: no longer R23.1, R24.2
- net MOTOR_L_CELL3: no longer R21.1, R22.2
- net MOTOR_R_CELL1: no longer R33.1, R34.2
- net MOTOR_R_CELL2: no longer R27.1, R28.2
- net MOTOR_R_CELL3: no longer R25.1, R26.2
- net N$1: no longer PCB_CELL2.3
- net N$11: now also CONV_SW_REG.2; no longer CONVPOW.1
- net N$14: no longer MOTOR_L_CELL3.2, R32.1
- net N$27: no longer PCB_CELL2.2, PCB_CELL3.3
- net N$41: no longer C15.2, C17.2, PCB_CELL2.1, PCB_CELL2.4, PCB_CELL3.1, PCB_CELL3.4, R18.1, R20.1, R29.2
- net N$43: no longer MOTOR_L_CELL2.3
- net N$45: no longer MOTOR_L_CELL2.2, MOTOR_L_CELL3.3
- net N$47: no longer C16.1, C5.1, MOTOR_L_CELL2.7, MOTOR_L_CELL3.7
- net N$50: no longer C16.2, C5.2, MOTOR_L_CELL2.1, MOTOR_L_CELL2.4, MOTOR_L_CELL3.1, MOTOR_L_CELL3.4, R22.1, R24.1, R31.2
- net N$53: no longer MOTOR_R_CELL2.3
- net N$54: no longer MOTOR_R_CELL3.2, R34.1
- net N$55: no longer MOTOR_R_CELL2.2, MOTOR_R_CELL3.3
- net N$57: no longer C19.1, C20.1, MOTOR_R_CELL2.7, MOTOR_R_CELL3.7
- net N$60: no longer C19.2, C20.2, MOTOR_R_CELL2.1, MOTOR_R_CELL2.4, MOTOR_R_CELL3.1, MOTOR_R_CELL3.4, R26.1, R28.1, R33.2
- net N$8: no longer PCB_CELL3.2, R30.1
- net PCB_CELL1: no longer R29.1, R30.2
- net PCB_CELL2: no longer R19.1, R20.2
- net PCB_CELL3: no longer R17.1, R18.2
- net PCB_IN: no longer C15.1, C17.1, PCB_CELL2.7, PCB_CELL3.7
- net VBAT: now also C23.1

Commit message: trying to finalize verion 1 of PCB
Parts:
- removed C23: 100uF, rcl:C1206
- removed C4, C6, C7, C8, C9: 22uF, rcl:C1206
- removed D2: 1N4446, diode:DO35-10
- removed GND, VDD: TEST-POINT3X4, SparkFun-Connectors:PAD.03X.04
- removed MOTOR_L_IN, MOTOR_L_OUT, MOTOR_R_IN, MOTOR_R_OUT, PCB_IN, PCB_OUT: (no value), PRT-10474:SHDR2W320P716_1X2_1574X813X158
- removed MOTOR_R_SENSE_IN: JST-XH-04-PIN-LONG-PAD, Rembrandt Electronics - JST XH Connectors v1-0:JST-XH-04-PACKAGE-LONG-PAD
- removed Q10, Q12, Q13, Q14, Q15: 2N3906, transistor-pnp:TO92
- added D1, D3: V60D45C-M3_I, V60D45C-M3_I:TO-263AC(SMPD)
- added ESP_DEBUG: (no value), con-lstb:MA08-1
- added GPS_DEBUG: (no value), con-lstb:MA06-1
- added JP4, JP5: (no value), jumper:JP2
- added LDR0, LDR1, LDR2, LDR3, LDR4, MOTOR_L_CELL1, MOTOR_L_CELL2, MOTOR_R_CELL1, MOTOR_R_CELL2, PCB_CELL1, PCB_CELL2: TPSQB2,54, testpad:B2,54
- added LED1: BLUE, led:CHIPLED_0805
- added MOTOR_L_CELL3, MOTOR_R_CELL3, PCB_CELL3: PCB_CELL3, testpad:B2,54
- added MOTOR_R_SENSE: MOTOR_R_SENSE_IN, bt_con-jst-xh:B4B-XH
- added PCB_SW: (no value), PRT-10474:SHDR2W320P716_1X2_1574X813X158
- added R17, R23, R29: 180k, resistor:R0805
- added R18, R24, R30: 6.2k, resistor:R0805
- added R19, R25, R31: 8.2k, resistor:R0805
- added R20, R26, R32: 5.1k, resistor:R0805
- added R21, R27, R33: 680, resistor:R0805
- added R22, R28, R34: 2.4k, resistor:R0805
- added R48: 200, rcl:R0805
- added R49: 10K, rcl:R0805
- added R50, R52: 100K, rcl:R0805
- added R51: 510, rcl:R0805
- added R53, R54, R55: 100k, resistor:R1206
- C1, C2, C3: value 22uF -> 100uF; device rcl:C1206 -> rcl:140CLH-0810
- C10: device rcl:C1206 -> resistor:C0805
- C18: value 100nF -> 22uF; device resistor:C1206 -> resistor:C0805
- C25, C26, C30, C31, C32, C33, C34, C35, C36, C37, C38, C39, C40, C41, C42, C43, C44, C45: device SparkFun-Capacitors:1206 -> resistor:C0805K
- MOTOR_L_SENSE_IN: value JST-XH-04-PIN-LONG-PAD -> MOTOR_L_SENSE_IN; device Rembrandt Electronics - JST XH Connectors v1-0:JST-XH-04-PACKAGE-LONG-PAD -> bt_con-jst-xh:B4B-XH
- MOTOR_L_SENSE_OUT, MOTOR_R_SENSE_OUT: value JST-XH-04-PIN-LONG-PAD -> MOTOR_R_SENSE_OUT; device Rembrandt Electronics - JST XH Connectors v1-0:JST-XH-04-PACKAGE-LONG-PAD -> bt_con-jst-xh:B4B-XH
- PCB_SENSE_IN: value JST-XH-04-PIN-LONG-PAD -> PCB_SENSE_IN; device Rembrandt Electronics - JST XH Connectors v1-0:JST-XH-04-PACKAGE-LONG-PAD -> bt_con-jst-xh:B4B-XH
- PCB_SENSE_OUT: value JST-XH-04-PIN-LONG-PAD -> PCB_SENSE_OUT; device Rembrandt Electronics - JST XH Connectors v1-0:JST-XH-04-PACKAGE-LONG-PAD -> bt_con-jst-xh:B4B-XH
- R1, R16, R2, R3, R4, R5, R6, R7, R8: device resistor:R1206 -> resistor:R0805
- R10, R9: device resistor:R0805 -> resistor:R1206
- R11, R12, R13, R14, R35, R36, R38: device resistor:R1206 -> rcl:R0805
- R15: value 10k -> 100k; device resistor:R1206 -> resistor:R0805
- R37, R40, R42, R46: value 2k -> 100k; device rcl:R1206 -> resistor:R1206
- R39, R41: value 1k -> 100k; device rcl:R1206 -> resistor:R1206
- R43: value 1k -> 1M; device rcl:R1206 -> resistor:R0805
- R44: value 2k -> 1M; device rcl:R1206 -> resistor:R0805
- R45: value 1k -> 200; device rcl:R1206 -> rcl:R0805
- R47: value 1k -> 10K; device rcl:R1206 -> rcl:R0805
- moved R46 283.5 mm to (-90.2, -130.8), flipped to the top
- moved R45 263.0 mm to (-83.8, -124.5)
- moved R47 211.7 mm to (-67.3, -68.6)
- moved R42 201.1 mm to (-66.0, -40.6), flipped to the top
- moved R40 195.9 mm to (-66.0, -27.9), flipped to the top
- moved R41 192.5 mm to (-66.0, -34.3)
- moved R37 191.1 mm to (-66.0, -15.2), flipped to the top
- moved R39 187.4 mm to (-66.0, -21.6)
- moved R43 108.1 mm to (55.9, 5.08), flipped to the bottom
- moved R44 91.0 mm to (43.2, 14.0), turned to 180 degrees
- moved MOTOR_R_SENSE_OUT 84.1 mm to (-35.6, 182.9)
- moved MOTOR_L_SENSE_OUT 68.7 mm to (-35.6, 203.2)
- moved R2 60.5 mm to (15.2, 12.7)
- moved R1 58.9 mm to (15.2, 7.62)
- moved R8 57.6 mm to (15.2, 12.7), flipped to the top
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Connections:
- removed net ADJ/GND: MICRO_REG.1
- removed net GDC: DCIN.1, DCOUT.1, SOLAR.1
- removed net N$40: PCB_SENSE_IN.4, PCB_SENSE_OUT.4
- removed net N$41: PCB_IN.1, PCB_OUT.1
- removed net N$53: MOTOR_R_SENSE_IN.3, MOTOR_R_SENSE_OUT.3
- removed net N$54: MOTOR_R_SENSE_IN.1, MOTOR_R_SENSE_OUT.1
- removed net N$55: MOTOR_R_SENSE_IN.2, MOTOR_R_SENSE_OUT.2
- removed net N$56: MOTOR_R_SENSE_IN.4, MOTOR_R_SENSE_OUT.4
- removed net N$57: MOTOR_R_IN.2, MOTOR_R_OUT.2
- removed net N$60: MOTOR_R_IN.1, MOTOR_R_OUT.1
- removed net N$64: BOOT0.2, R36.2
- removed net N$74: LDR_HEADER.2, Q10.2, R37.2
- removed net N$76: LDR_HEADER.8, Q15.2, R46.2
- removed net N$77: LDR_HEADER.4, Q12.2, R40.2
- removed net N$79: LDR_HEADER.6, Q13.2, R42.2
- removed net N$85: LDR_HEADER.10, Q14.2, R44.2
- removed net PCB_IN: PCB_IN.2, PCB_OUT.2
- removed net VDC: D2.C, DCIN.2, DCOUT.2
- new net N$10: MOTOR_L_SENSE_IN.P$3, MOTOR_L_SENSE_OUT.P$3, R27.1
- new net N$12: MOTOR_L_SENSE_IN.P$2, MOTOR_L_SENSE_OUT.P$2, R25.1
- new net N$17: MOTOR_R_SENSE.P$3, MOTOR_R_SENSE_OUT.P$3, R33.1
- new net N$20: MOTOR_R_SENSE.P$2, MOTOR_R_SENSE_OUT.P$2, R31.1
- new net N$28: MOTOR_R_SENSE.P$1, MOTOR_R_SENSE_OUT.P$1, R29.1
- new net N$35: D1.3, D3.3, DCOUT.2
- new net N$4: D1.1, D1.2, DCIN.2
- new net N$48: ESP8266_HEADER.4, ESP8266_HEADER.8, JP4.2
- new net N$49: GPS_HEADER.1, JP5.3
- new net N$51: LASER_HEADER.1, LASER_HEADER.3, LASER_HEADER.5, LASER_HEADER.7, LASER_HEADER.9, LASR_SW.D
- new net N$52: PCBPOWER.2, PCB_SW.1
- net CMP_SCL: now also R47.1
- net CMP_SDA: now also R49.1
- net ESP_GPIO0: now also ESP_DEBUG.8
- net ESP_GPIO2: now also ESP_DEBUG.7, R50.1
- net ESP_RX: now also ESP_DEBUG.4
- net ESP_TX: now also ESP_DEBUG.5
- net GND: now also C1.-, C2.-, C3.-, C45.2, DCIN.1, DCOUT.1, ESP_DEBUG.1, GPS_DEBUG.1, LED1.C, MICRO_REG.1, MOTOR_L_SENSE_IN.P$4, MOTOR_L_SENSE_OUT.P$4, MOTOR_R_SENSE.P$4, MOTOR_R_SENSE_OUT.P$4, PCB_SENSE_IN.P$4, PCB_SENSE_OUT.P$4, R18.2, R20.2, R22.2, R24.2, R26.2, R28.2, R30.2, R32.2, R34.2, R51.2, RASPI_SW.S, SOLAR.1; no longer C1.2, C2.2, C23.2, C3.2, C4.2, C45.1, C6.2, C7.2, C8.2, C9.2, GND.P$1, LASER_HEADER.1, LASER_HEADER.3, LASER_HEADER.5, LASER_HEADER.7, LASER_HEADER.9, R15.1, R37.1, R39.1, R40.1, R41.1, R42.1, R43.1, R44.1, R45.1, R46.1, R47.1, RASPI_SW.D
- net GPS_RX: now also GPS_DEBUG.4
- net GPS_TX: now also GPS_DEBUG.5
- net LASER_MOS: now also R55.1
- net LDR0: now also LDR0.TP, LDR_HEADER.2, R37.1; no longer Q10.1, R39.2
- net LDR1: now also LDR1.TP, LDR_HEADER.4, R39.1; no longer Q12.1, R41.2
- net LDR2: now also LDR2.TP, LDR_HEADER.6, R40.1; no longer Q13.1, R43.2
- net LDR3: now also LDR3.TP, LDR_HEADER.8, R41.1; no longer Q15.1, R47.2
- net LDR4: now also LDR4.TP, LDR_HEADER.10, R42.1; no longer Q14.1, R45.2
- net LDR_MOS: now also R54.1
- net L_MOS: now also R46.2
- net MOTOR_L_CELL1: now also MOTOR_L_CELL1.TP, R27.2, R28.1
- net MOTOR_L_CELL2: now also MOTOR_L_CELL2.TP, R25.2, R26.1
- net MOTOR_L_CELL3: now also MOTOR_L_CELL3.TP, R23.2, R24.1
- net MOTOR_R_CELL1: now also MOTOR_R_CELL1.TP, R33.2, R34.1
- net MOTOR_R_CELL2: now also MOTOR_R_CELL2.TP, R31.2, R32.1
- net MOTOR_R_CELL3: now also MOTOR_R_CELL3.TP, R29.2, R30.1
- net N$1: now also PCB_SENSE_IN.P$3, PCB_SENSE_OUT.P$3, R21.1; no longer PCB_SENSE_IN.3, PCB_SENSE_OUT.3
- net N$11: now also R43.2
- net N$14: now also MOTOR_L_SENSE_IN.P$1, MOTOR_L_SENSE_OUT.P$1, R23.1; no longer MOTOR_L_SENSE_IN.1, MOTOR_L_SENSE_OUT.1
- net N$16: now also C2.+; no longer C6.1
- net N$19: now also R44.2, RASPI_SW.D; no longer RASPI_SW.S
- net N$2: no longer C9.1
- net N$27: now also PCB_SENSE_IN.P$2, PCB_SENSE_OUT.P$2, R19.1; no longer PCB_SENSE_IN.2, PCB_SENSE_OUT.2
- net N$43: now also IC5.62, R45.1; no longer MOTOR_L_SENSE_IN.3, MOTOR_L_SENSE_OUT.3
- net N$44: now also R52.2
- net N$45: now also BOOT0.2, R51.1; no longer MOTOR_L_SENSE_IN.2, MOTOR_L_SENSE_OUT.2
- net N$46: now also GPS_DEBUG.3, JP5.1; no longer MOTOR_L_SENSE_IN.4, MOTOR_L_SENSE_OUT.4
- net N$47: now also LDR_SW.D, R37.2, R39.2, R40.2, R41.2, R42.2; no longer MOTOR_L_IN.2, MOTOR_L_OUT.2
- net N$5: now also D3.1, D3.2; no longer D2.A
- net N$50: now also LED1.A, R45.2; no longer MOTOR_L_IN.1, MOTOR_L_OUT.1
- net N$6: now also C1.+; no longer C7.1
- net N$69: now also BOOT0.1
- net N$71: now also R46.1
- net N$72: now also R53.1
- net N$8: now also PCB_SENSE_IN.P$1, PCB_SENSE_OUT.P$1, R17.1; no longer PCB_SENSE_IN.1, PCB_SENSE_OUT.1
- net N$9: no longer LTE_PWR.2
- net PCB_CELL1: now also PCB_CELL1.TP, R21.2, R22.1
- net PCB_CELL2: now also PCB_CELL2.TP, R19.2, R20.1
- net PCB_CELL3: now also PCB_CELL3.TP, R17.2, R18.1
- net R_MOS: now also R53.2
- net VBAT: now also PCB_SW.2, R15.1, R43.1, R44.1; no longer C1.1, C2.1, C23.1, C3.1, C4.1, PCBPOWER.2
- net VCC: now also C45.1, ESP_DEBUG.3, JP4.1, JP4.3, JP5.2, R36.2, R47.2, R48.1, R48.2, R49.2, R50.2, R52.1, R54.2, R55.2; no longer BOOT0.1, C45.2, ESP8266_HEADER.4, ESP8266_HEADER.8, GPS_HEADER.1, VDD.P$1
- net VDD: now also C3.+; no longer C8.1, LASR_SW.D, LDR_SW.D, Q10.3, Q12.3, Q13.3, Q14.3, Q15.3

Commit message: update
Parts:
- removed C24: 100nF, SparkFun-Capacitors:1206
- removed C36, C37: 100nF, resistor:C0805K
- removed MOTOR_L_CELL1, MOTOR_L_CELL2, MOTOR_R_CELL1, MOTOR_R_CELL2, PCB_CELL1, PCB_CELL2: TPSQB2,54, testpad:B2,54
- removed MOTOR_L_CELL3, MOTOR_R_CELL3, PCB_CELL3: PCB_CELL3, testpad:B2,54
- removed MOTOR_R_SENSE: MOTOR_R_SENSE_IN, bt_con-jst-xh:B4B-XH
- added C4: 100uF, rcl:140CLH-0810
- added C5: 100nF, rcl:C0805
- added L_CELL1, L_CELL2, PCB1, PCB2, R_CELL1, R_CELL2: TPSQB2,54, testpad:B2,54
- added L_CELL3, PCB3, R_CELL3: PCB_CELL3, testpad:B2,54
- added MOTOR_R_SENSE_IN: MOTOR_R_SENSE_IN, bt_con-jst-xh:B4B-XH
- added R56: 200, rcl:R0805
- BOOT0, NRST: value (none) -> IRF512; device zetex:SOT-23 -> transistor-power:TO220BV
- C25, C26, C30, C32, C33, C34, C38, C39, C40, C41, C42, C43, C44, C45: device resistor:C0805K -> rcl:C0805
- C31: value 1uF -> 100nF; device resistor:C0805K -> rcl:C0805
- C35: value 100nF -> 1uF; device resistor:C0805K -> rcl:C0805
- moved LDR0 387.4 mm to (61.0, 106.7), turned to 180 degrees
- moved LDR1 376.9 mm to (61.0, 101.6), turned to 180 degrees
- moved LDR2 366.5 mm to (61.0, 96.5), turned to 180 degrees
- moved LDR3 356.2 mm to (61.0, 91.4), turned to 180 degrees
- moved LDR4 345.9 mm to (61.0, 86.4), turned to 180 degrees
- moved R55 312.6 mm to (68.6, 119.4)
- moved R53 301.4 mm to (57.1, 125.7), flipped to the bottom, turned to 90 degrees
- moved R46 284.9 mm to (57.1, 113.0), flipped to the bottom, turned to 90 degrees
- moved PCB_SW 281.0 mm to (60.2, 22.0), turned to 90 degrees
- moved R54 271.1 mm to (68.6, 76.2)
- moved JP5 241.6 mm to (72.4, 71.1)
- moved LED1 237.2 mm to (33.8, 76.5), turned to 180 degrees
- moved R45 236.2 mm to (33.8, 80.4), turned to 270 degrees
- moved R52 228.8 mm to (22.6, 116.5), turned to 90 degrees
- moved GPS_DEBUG 225.0 mm to (66.0, 63.5), turned to 90 degrees
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Connections:
- removed net ESP_RST: ESP8266_HEADER.6
- removed net N$180: C30.1, C35.1, IC5.21, IC5.22, R11.1
- new net N$37: PWR.A, R48.2
- new net N$39: C30.1, C35.1, IC5.21, R11.1
- new net N$40: C31.1, C34.1, IC5.22, L1.1, R11.2
- new net N$41: ESP_DEBUG.3, JP4.3
- net ESP_GPIO2: now also BOOT0.G; no longer BOOT0.3
- net GND: now also C31.2, C34.2, C4.-, C5.2, CON_SW.S, MOTOR_R_SENSE_IN.P$4, NRST.S, R15.1; no longer C24.1, C31.1, C34.1, C36.2, C37.2, CON_SW.D, MOTOR_R_SENSE.P$4, NRST.2, R16.1
- net MOTOR_L_CELL1: now also L_CELL1.TP; no longer MOTOR_L_CELL1.TP
- net MOTOR_L_CELL2: now also L_CELL2.TP; no longer MOTOR_L_CELL2.TP
- net MOTOR_L_CELL3: now also L_CELL3.TP; no longer MOTOR_L_CELL3.TP
- net MOTOR_R_CELL1: now also R_CELL1.TP; no longer MOTOR_R_CELL1.TP
- net MOTOR_R_CELL2: now also R_CELL2.TP; no longer MOTOR_R_CELL2.TP
- net MOTOR_R_CELL3: now also R_CELL3.TP; no longer MOTOR_R_CELL3.TP
- net N$11: now also CON_SW.D; no longer CON_SW.S
- net N$17: now also MOTOR_R_SENSE_IN.P$3; no longer MOTOR_R_SENSE.P$3
- net N$20: now also MOTOR_R_SENSE_IN.P$2; no longer MOTOR_R_SENSE.P$2
- net N$28: now also MOTOR_R_SENSE_IN.P$1; no longer MOTOR_R_SENSE.P$1
- net N$34: now also R56.1, RST.A; no longer C31.2, C34.2, C36.1, C37.1, L1.1, R11.2
- net N$44: now also NRST.G; no longer NRST.3
- net N$45: now also BOOT0.S; no longer BOOT0.2
- net N$63: now also C5.1, R56.2; no longer C24.2, RST.A
- net N$69: now also BOOT0.D; no longer BOOT0.1
- net N$9: now also LTE_PWR.2
- net NRST: now also NRST.D; no longer NRST.1
- net PCB_CELL1: now also PCB1.TP; no longer PCB_CELL1.TP
- net PCB_CELL2: now also PCB2.TP; no longer PCB_CELL2.TP
- net PCB_CELL3: now also PCB3.TP; no longer PCB_CELL3.TP
- net VBAT: now also R16.1; no longer R15.1
- net VCC: now also C4.+; no longer ESP_DEBUG.3, JP4.3, PWR.A, R48.2
Routing:
- net VCC: track 0.00 -> 539.2 mm, vias 0 -> 33
- net VDD: track 0.00 -> 126.5 mm, vias 0 -> 4
- net ESP_GPIO0: track 0.00 -> 104.0 mm, vias 0 -> 6
- net VBAT: track 0.00 -> 98.8 mm, vias 0 -> 1
- net ESP_RX: track 0.00 -> 75.8 mm, vias 0 -> 5
- net CMP_SCL: track 0.00 -> 73.5 mm, vias 0 -> 3
- net CMP_SDA: track 0.00 -> 65.9 mm, vias 0 -> 3
- net ESP_TX: track 0.00 -> 58.5 mm, vias 0 -> 2
- net CMP_MOSI: track 0.00 -> 55.0 mm, vias 0 -> 2
- net CMP_INT: track 0.00 -> 52.9 mm, vias 0 -> 2
- net ESP_GPIO2: track 0.00 -> 52.6 mm, vias 0 -> 3
- net CMP_SCLK: track 0.00 -> 52.1 mm, vias 0 -> 2
- net NRST: track 0.00 -> 50.8 mm, vias 0 -> 2
- net CMP_MISO: track 0.00 -> 50.5 mm, vias 0 -> 2
- net N$16: track 0.00 -> 49.3 mm, vias 0 -> 2
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- added copper zone on layer 1, net GND
- added copper zone on layer 16, net GND
- added copper zone on layer 1, net N$35
- added copper zone on layer 1, net N$4
- added copper zone on layer 1, net N$5
Other:
- board size 78.7 x 272.7 mm -> 78.7 x 194 mm

Commit message: revised
Parts:
- moved LED1 14.8 mm to (46.5, 68.8)
- moved R45 13.7 mm to (46.5, 75.3)
- moved R46 7.62 mm to (49.5, 113.0)
- moved R53 7.62 mm to (49.5, 125.7)
- moved CMP_BRKOUT 3.81 mm to (10.2, 176.5)
- moved C45 3.39 mm to (43.9, 97.3)
- moved C12 1.27 mm to (26.7, 177.8)
- moved R9 0.40 mm to (25.5, 173.6)
- moved C21 0.40 mm to (20.4, 173.6)
- moved C30 0.38 mm to (29.1, 95.5)
- moved C35 0.38 mm to (29.1, 93.5)
- moved C13 0.28 mm to (7.49, 110.7)
- moved C42 0.25 mm to (24.8, 95.0)
- moved R18 0.25 mm to (50.8, 63.2)
- moved R20 0.25 mm to (54.6, 63.2)
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Connections:
- removed net N$18: C11.1, CMP_BRKOUT.1, IC3.11, IC3.12, IC3.15
- removed net N$31: CMP_BRKOUT.5, IC3.10
- removed net N$32: C12.2, CMP_BRKOUT.7, IC3.9
- removed net N$33: C21.1, CMP_BRKOUT.9, IC3.4
- net N$21: now also C12.2, C21.1, CMP_BRKOUT.5, CMP_BRKOUT.7, CMP_BRKOUT.9, IC3.10, IC3.4, IC3.9
- net N$30: now also C11.1, CMP_BRKOUT.1, IC3.11, IC3.12, IC3.15
Routing:
- net N$30: track 0.00 -> 108.4 mm, vias 0 -> 7
- net GND: track 0.00 -> 106.0 mm, vias 2 -> 22
- net R_PWM: track 0.00 -> 103.9 mm, vias 0 -> 3
- net L_PWM: track 0.00 -> 95.7 mm, vias 0 -> 3
- net C_MOS: track 3.08 -> 95.2 mm, vias 0 -> 3
- net PCB_CELL1: track 5.08 -> 90.1 mm, vias 1 -> 4
- net RASPI_MOS: track 3.93 -> 87.1 mm, vias 0 -> 3
- net MOTOR_R_CELL2: track 5.08 -> 84.6 mm, vias 1 -> 5
- net MOTOR_L_CELL2: track 4.13 -> 81.1 mm, vias 1 -> 7
- net PCB_CELL3: track 5.08 -> 81.8 mm, vias 1 -> 4
- net PCB_CELL2: track 5.08 -> 79.0 mm, vias 1 -> 7
- net MOTOR_L_CELL3: track 5.08 -> 77.2 mm, vias 1 -> 7
- net L_MOS: track 0.00 -> 70.2 mm, vias 0 -> 3
- net LASER_MOS: track 0.00 -> 69.9 mm, vias 0 -> 4
- net R_MOS: track 0.00 -> 66.9 mm, vias 0 -> 3
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- added copper zone on layer 1, net N$21

Commit message: update
Parts:
- moved R50 0.51 mm to (28.2, 71.1), turned to 180 degrees
Connections:
- removed net N$71: LEFT_MOTOR.5, LM_SW.S, R46.1
- removed net N$72: R53.1, RIGHT_MOTOR.5, RM_SW.S
- net ESP_GPIO2: now also R50.2; no longer R50.1
- net GND: now also LEFT_MOTOR.5, LM_SW.S, R46.1, R50.1, R53.1, RIGHT_MOTOR.5, RM_SW.S
- net VCC: no longer R50.2
Routing:
- net N$71: track 31.1 -> 0.00 mm, vias 2 -> 0
- net N$72: track 26.5 -> 0.00 mm
- net ESP_RX: track 75.3 -> 63.8 mm, vias 7 -> 2
- net N$30: track 108.4 -> 98.1 mm
- net VCC: track 571.6 -> 563.8 mm, vias 36 -> 33
- net N$26: track 27.9 -> 20.5 mm, vias 2 -> 0
- net N$48: track 20.0 -> 15.0 mm, vias 3 -> 0
- net CMP_SDA: track 66.0 -> 61.1 mm
- net N$41: track 17.8 -> 13.3 mm, vias 2 -> 0
- net GND: track 106.0 -> 102.3 mm, vias 22 -> 21
- net ESP_GPIO0: track 104.0 -> 100.2 mm, vias 6 -> 4
- net CMP_SCL: track 74.7 -> 71.9 mm, vias 5 -> 3
- net ESP_GPIO2: track 52.6 -> 55.0 mm, vias 3 -> 1
- net PCB_CELL2: track 79.0 -> 76.8 mm, vias 7 -> 3
- net LDR2: track 43.9 -> 41.7 mm, vias 4 -> 2
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Other:
- board text added: "ECE477 Group 6 Qianli Ma Shuang Liu Tianjie Jia Peiyuan Shen Version 1 Modified 10.9.2018"

Commit message: update
Parts:
- moved C11 2.54 mm to (24.1, 179.1)
- moved C12 2.54 mm to (26.7, 175.3)
- moved C21 2.54 mm to (20.4, 171.1)
- moved IC3 2.54 mm to (21.6, 175.3)
- moved R9 2.54 mm to (25.5, 171.1)
- moved Q11 2.54 mm to (34.0, 107.2)
- moved C22 2.54 mm to (16.5, 176.5)
- moved CMP_BRKOUT 2.54 mm to (10.2, 174.0)
- moved R10 2.54 mm to (16.5, 176.5)
- moved C39 1.27 mm to (30.5, 110.5)
- moved C40 1.27 mm to (36.8, 110.5)
- moved R38 1.27 mm to (33.3, 103.5), flipped to the top, turned to 180 degrees
Connections:
- net N$21 renamed GND_BREAKOUT
- net N$30 renamed VDD_BREAKOUT
Routing:
- net GND: track 102.3 -> 111.9 mm, vias 21 -> 19
- net MOTOR_R_CELL1: track 64.1 -> 56.8 mm
- net LDR1: track 45.8 -> 41.5 mm
- net GND_BREAKOUT: track 7.62 -> 5.08 mm
- net N$70: track 11.4 -> 13.2 mm
- net LDR2: track 41.7 -> 43.1 mm
- net N$65: track 3.48 -> 4.49 mm, vias 1 -> 0
- net LDR4: track 47.8 -> 47.0 mm
- net LDR0: track 42.9 -> 42.3 mm
- net VCC: track 563.8 -> 564.4 mm
Other:
- board size 78.7 x 194 mm -> 78.7 x 186.4 mm

Commit message: ready for submission
Parts:
- added C15, C16, C17, C19, C20, C6, C7, C8, C9: 22nF, eagle-ltspice:C0805
- R17, R23, R29: value 180k -> 18k
- moved R27 5.08 mm to (43.3, 53.3)
- moved R17 5.08 mm to (50.8, 53.3)
- moved R19 5.08 mm to (54.6, 53.3)
- moved R21 5.08 mm to (58.4, 53.3)
- moved R23 5.08 mm to (35.6, 53.3)
- moved R25 5.08 mm to (39.4, 53.3)
- moved R29 3.81 mm to (50.8, 68.6), turned to 90 degrees
- moved R31 3.81 mm to (54.6, 68.6), turned to 90 degrees
- moved R33 3.81 mm to (58.4, 68.6), turned to 90 degrees
Connections:
- net GND: now also C15.2, C16.2, C17.2, C19.2, C20.2, C6.2, C7.2, C8.2, C9.2
- net MOTOR_L_CELL1: now also C16.1
- net MOTOR_L_CELL2: now also C15.1
- net MOTOR_L_CELL3: now also C9.1
- net MOTOR_R_CELL1: now also C20.1
- net MOTOR_R_CELL2: now also C19.1
- net MOTOR_R_CELL3: now also C17.1
- net PCB_CELL1: now also C8.1
- net PCB_CELL2: now also C7.1
- net PCB_CELL3: now also C6.1
Routing:
- net GND: track 111.9 -> 410.4 mm
- net MOTOR_R_CELL2: track 83.9 -> 57.8 mm, vias 5 -> 3
- net MOTOR_R_CELL3: track 50.6 -> 68.6 mm, vias 4 -> 3
- net CMP_SCL: track 71.9 -> 62.5 mm
- net PCB_CELL2: track 76.8 -> 85.9 mm, vias 3 -> 2
- net N$14: track 20.2 -> 11.8 mm, vias 1 -> 0
- net MOTOR_L_CELL3: track 77.2 -> 69.1 mm, vias 7 -> 5
- net PCB_CELL1: track 89.1 -> 81.3 mm
- net SWDIO: track 64.2 -> 57.0 mm
- net GPS_RX: track 60.0 -> 53.3 mm, vias 3 -> 2
- net N$20: track 35.0 -> 28.6 mm
- net N$17: track 35.0 -> 28.9 mm
- net N$10: track 17.9 -> 12.9 mm, vias 1 -> 0
- net N$12: track 17.4 -> 12.3 mm, vias 1 -> 0
- net N$28: track 35.3 -> 30.4 mm
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Other:
- board text added: "ECE477 Group 6 Qianli Ma Shuang Liu Tianjie Jia Peiyuan Shen Version 1 Modified 10.18.2018"
- board text removed: "ECE477 Group 6 Qianli Ma Shuang Liu Tianjie Jia Peiyuan Shen Version 1 Modified 10.9.2018"
